File: backplane-boards/backplane-breakout-big/LED_Driver.sch (KiCad schematic (older format))
At the start: 26 parts, among them Q600 BC857AW,115, Q601 BC857AW,115, Q602 BC857AW,115, Q603 BC847CW,115, U600 TLC59282, U601 TLC59282

Commit message: breakout-big
Parts:
- removed Q600, Q601, Q602: BC857AW,115, Package_TO_SOT_SMD:SOT-323_SC-70, symbol Device:Q_PNP_BEC
- removed Q603: BC847CW,115, Package_TO_SOT_SMD:SOT-323_SC-70, symbol Device:Q_NPN_BEC
- removed R602, R603, R604: 0R, Resistor_SMD:R_0603_1608Metric, symbol Device:R_US
- removed R605, R606, R607, R609: 4.7k, Resistor_SMD:R_0402_1005Metric, symbol Device:R_US
- removed R608: 10k, Resistor_SMD:R_0402_1005Metric, symbol Device:R_US
- D600_1, D600_8: footprint CubeSat_Backplane:156125M173000 -> backplane-breakout-big:156125M173000
- D600_2: renamed from D600_5; footprint CubeSat_Backplane:156125M173000 -> backplane-breakout-big:156125M173000
- D600_3: renamed from D600_2; footprint CubeSat_Backplane:156125M173000 -> backplane-breakout-big:156125M173000
- D600_4: renamed from D600_6; footprint CubeSat_Backplane:156125M173000 -> backplane-breakout-big:156125M173000
- D600_5: renamed from D600_3; footprint CubeSat_Backplane:156125M173000 -> backplane-breakout-big:156125M173000
- D600_6: renamed from D600_7; footprint CubeSat_Backplane:156125M173000 -> backplane-breakout-big:156125M173000
- D600_7: renamed from D600_4; footprint CubeSat_Backplane:156125M173000 -> backplane-breakout-big:156125M173000
- U1: renamed from U600; symbol CubeSat_Backplane:TLC59282 -> backplane-breakout-big:TLC59282
- U2: renamed from U601; symbol CubeSat_Backplane:TLC59282 -> backplane-breakout-big:TLC59282
- renumbered C600 to C1, C601 to C2, R600 to R40, R601 to R41
Connections:
- net labels added: 5V_DEBUG, SOUT
- net labels removed: 5V_USB, SCLK_LED, SIN_LED, SOUT_LED_1, ~enable
- wire segments 116 -> 92
Other:
- note removed: "Only allows data lines to pass thru if 5vusb is connected\ndisconects these devices in flight"
