File: backplane-boards/backplane-breakout-big/backplane-breaout-big.sch (KiCad schematic (older format))
At the start: 2 parts, among them J1 Breakout Connector, J2 Breakout Connector

Commit message: breakout-big
Parts:
- added D1, D10, D2, D3, D5, D7, D8, D9: GREEN, LED_SMD:LED_0603_1608Metric_Castellated, symbol Device:LED
- added D11, D12, D4, D6: ORANGE, LED_SMD:LED_0603_1608Metric_Castellated, symbol Device:LED
- added D13, D14, D20, D22: BLUE, LED_SMD:LED_0603_1608Metric_Castellated, symbol Device:LED
- added D15, D16, D17, D18, D19, D21, D23: RED, LED_SMD:LED_0603_1608Metric_Castellated, symbol Device:LED
- added J10: -Z_SOLAR_RTN, backplane-breakout-big:Keystone_476, symbol Connector_Generic:Conn_01x01
- added J11: +Y_SOLAR_PWR, backplane-breakout-big:Keystone_476, symbol Connector_Generic:Conn_01x01
- added J12: +Y_SOLAR_RTN, backplane-breakout-big:Keystone_476, symbol Connector_Generic:Conn_01x01
- added J13: -X_SOLAR_PWR, backplane-breakout-big:Keystone_476, symbol Connector_Generic:Conn_01x01
- added J14: -X_SOLAR_RTN, backplane-breakout-big:Keystone_476, symbol Connector_Generic:Conn_01x01
- added J15: 3.3V_SYS, backplane-breakout-big:Keystone_476, symbol Connector_Generic:Conn_01x01
- added J16: +5V_SYS, backplane-breakout-big:Keystone_476, symbol Connector_Generic:Conn_01x01
- added J17: VCC_RF, backplane-breakout-big:Keystone_476, symbol Connector_Generic:Conn_01x01
- added J18: 5V_DEBUG, backplane-breakout-big:Keystone_476, symbol Connector_Generic:Conn_01x01
- added J19: GND, backplane-breakout-big:Keystone_476, symbol Connector_Generic:Conn_01x01
- added J20, J24: Conn_02x04_Odd_Even, symbol Connector_Generic:Conn_02x04_Odd_Even
- added J200_1: HSEC8-160-01-S-DV-A-K-TR, backplane-breakout-big:HSEC8-160-01-S-DV-A-K-TR, symbol backplane-breakout-big:Conn_02x60_Top_Bottom
- added J21: AGND, backplane-breakout-big:Keystone_476, symbol Connector_Generic:Conn_01x01
- added J22, J23: Conn_02x30_Odd_Even, Connector_PinHeader_2.54mm:PinHeader_2x30_P2.54mm_Vertical, symbol Connector_Generic:Conn_02x30_Odd_Even
- added J3: DEBUG POWER SEND JUMPER, symbol Connector_Generic:Conn_01x02
- added J4: PACK+, backplane-breakout-big:Keystone_476, symbol Connector_Generic:Conn_01x01
- added J5: Conn_01x08, symbol Connector_Generic:Conn_01x08
- added J6: PACK-, backplane-breakout-big:Keystone_476, symbol Connector_Generic:Conn_01x01
- added J7: +X_SOLAR_PWR, backplane-breakout-big:Keystone_476, symbol Connector_Generic:Conn_01x01
- added J8: +X_SOLAR_RTN, backplane-breakout-big:Keystone_476, symbol Connector_Generic:Conn_01x01
- added J9: -Z_SOLAR_PWR, backplane-breakout-big:Keystone_476, symbol Connector_Generic:Conn_01x01
- added Q1, Q10, Q11, Q12, Q18, Q19, Q2, Q22, Q23, Q3, Q4, Q5, Q6, Q7, Q8, Q9: DMG1012UW-7, Package_TO_SOT_SMD:SOT-323_SC-70, symbol Device:Q_NMOS_GSD
- added Q13, Q14, Q15, Q16, Q17, Q20, Q21: BSS84W-7-F, Package_TO_SOT_SMD:SOT-323_SC-70, symbol Device:Q_PMOS_GSD
- added R1, R13, R14, R15, R16, R17, R18, R2, R25, R26, R27, R28, R29, R3, R30, R31, R34, R35, R36, R37, R4, R5, R6: 1k, symbol Device:R_US
- added R10, R11, R12, R19, R20, R21, R22, R23, R24, R32, R33, R38, R39, R7, R8, R9: 10k, symbol Device:R_US
- added SW1: SEP1, backplane-breakout-big:SW_OS102011MS2QN1, symbol Switch:SW_SPDT
- added SW2: SEP2, backplane-breakout-big:SW_OS102011MS2QN1, symbol Switch:SW_SPDT
- added SW3: SEP3, backplane-breakout-big:SW_OS102011MS2QN1, symbol Switch:SW_SPDT
- added SW4: SEP4, backplane-breakout-big:SW_OS102011MS2QN1, symbol Switch:SW_SPDT
- added SW5: RBF, backplane-breakout-big:SW_OS102011MS2QN1, symbol Switch:SW_SPDT
- added SW6: USER_SW_1, backplane-breakout-big:SW_OS102011MS2QN1, symbol Switch:SW_SPDT
- added SW7: USER_SW_2, backplane-breakout-big:SW_OS102011MS2QN1, symbol Switch:SW_SPDT
- added SW8: USER_SW_3, backplane-breakout-big:SW_OS102011MS2QN1, symbol Switch:SW_SPDT
- added SW9: USER_SW_4, backplane-breakout-big:SW_OS102011MS2QN1, symbol Switch:SW_SPDT
- added TP1: SEP1, symbol Connector:TestPoint_Small
- added TP10: H1-2, symbol Connector:TestPoint_Small
- added TP100: H2-46, symbol Connector:TestPoint_Small
- added TP101: SELF_TEST (H1-47), symbol Connector:TestPoint_Small
- added TP102: USER_1 (H1-48), symbol Connector:TestPoint_Small
- added TP103: GND (H2-47), symbol Connector:TestPoint_Small
- added TP104: GND (H2-48), symbol Connector:TestPoint_Small
- added TP105: USER_2 (H1-49), symbol Connector:TestPoint_Small
- added TP106: USER_3 (H1-50), symbol Connector:TestPoint_Small
- added TP107: VBATT- (H2-49), symbol Connector:TestPoint_Small
- added TP108: VBATT- (H2-50), symbol Connector:TestPoint_Small
- added TP109: USER_4 (H1-51), symbol Connector:TestPoint_Small
- added TP11: H2-1, symbol Connector:TestPoint_Small
- added TP110: USER_5 (H1-52), symbol Connector:TestPoint_Small
- added TP111: USER_10 (H2-51), symbol Connector:TestPoint_Small
- added TP112: USER_11 (H2-52), symbol Connector:TestPoint_Small
- added TP113: +Y_SOLAR_TLE, symbol Connector:TestPoint_Small
- added TP114: -X_SOLAR_TLE, symbol Connector:TestPoint_Small
- added TP115: +Y_SOLAR_RTN, symbol Connector:TestPoint_Small
- added TP116: -X_SOLAR_RTN, symbol Connector:TestPoint_Small
- added TP117: +Y_SOLAR_PWR, symbol Connector:TestPoint_Small
- added TP118: -X_SOLAR_PWR, symbol Connector:TestPoint_Small
- added TP119: SEP3, symbol Connector:TestPoint_Small
- added TP12: H2-2, symbol Connector:TestPoint_Small
- added TP120: SEP4, symbol Connector:TestPoint_Small
- added TP13: H1-3, symbol Connector:TestPoint_Small
- added TP14: H1-4, symbol Connector:TestPoint_Small
- added TP15: H2-3, symbol Connector:TestPoint_Small
- added TP16: H2-4, symbol Connector:TestPoint_Small
- added TP17: H1-5, symbol Connector:TestPoint_Small
- added TP18: H1-6, symbol Connector:TestPoint_Small
- added TP19: H2-5, symbol Connector:TestPoint_Small
- added TP2: SEP2, symbol Connector:TestPoint_Small
- added TP20: H2-6, symbol Connector:TestPoint_Small
- added TP21: H1-7, symbol Connector:TestPoint_Small
- added TP22: H1-8, symbol Connector:TestPoint_Small
- added TP23: H2-7, symbol Connector:TestPoint_Small
- added TP24: H2-8, symbol Connector:TestPoint_Small
- added TP25: H1-9, symbol Connector:TestPoint_Small
- added TP26: H1-10, symbol Connector:TestPoint_Small
- added TP27: H2-0, symbol Connector:TestPoint_Small
- added TP28: H2-10, symbol Connector:TestPoint_Small
- added TP29: H1-11, symbol Connector:TestPoint_Small
- added TP3: -Z_SOLAR_TLE, symbol Connector:TestPoint_Small
- added TP30: H1-12, symbol Connector:TestPoint_Small
- added TP31: H2-11, symbol Connector:TestPoint_Small
- added TP32: H2-12, symbol Connector:TestPoint_Small
- added TP33: H1-13, symbol Connector:TestPoint_Small
- added TP34: H1-14, symbol Connector:TestPoint_Small
- added TP35: H2-13, symbol Connector:TestPoint_Small
- added TP36: H2-14, symbol Connector:TestPoint_Small
- added TP37: RBF (H1-15), symbol Connector:TestPoint_Small
- added TP38: H1-16, symbol Connector:TestPoint_Small
- added TP39: H2-15, symbol Connector:TestPoint_Small
- added TP4: +X_SOLAR_TLE, symbol Connector:TestPoint_Small
- added TP40: H2-16, symbol Connector:TestPoint_Small
- added TP41: H1-17, symbol Connector:TestPoint_Small
- added TP42: H1-18, symbol Connector:TestPoint_Small
- added TP43: H2-17, symbol Connector:TestPoint_Small
- added TP44: H2-18, symbol Connector:TestPoint_Small
- added TP45: H1-19, symbol Connector:TestPoint_Small
- added TP46: H1-20, symbol Connector:TestPoint_Small
- added TP47: H2-19, symbol Connector:TestPoint_Small
- added TP48: H2-20, symbol Connector:TestPoint_Small
- added TP49: H1-21, symbol Connector:TestPoint_Small
- added TP5: -Z_SOLAR_RTN, symbol Connector:TestPoint_Small
- added TP50: H1-22, symbol Connector:TestPoint_Small
- added TP51: H2-21, symbol Connector:TestPoint_Small
- added TP52: H2-22, symbol Connector:TestPoint_Small
- added TP53: H1-23, symbol Connector:TestPoint_Small
- added TP54: H1-24, symbol Connector:TestPoint_Small
- added TP55: H2-23, symbol Connector:TestPoint_Small
- added TP56: H2-24, symbol Connector:TestPoint_Small
- added TP57: H1-25, symbol Connector:TestPoint_Small
- added TP58: H1-26, symbol Connector:TestPoint_Small
- added TP59: 5V_SYS (H2-25), symbol Connector:TestPoint_Small
- added TP6: +X_SOLAR_RTN, symbol Connector:TestPoint_Small
- added TP60: 5V_SYS (H2-26), symbol Connector:TestPoint_Small
- added TP61: H1-27, symbol Connector:TestPoint_Small
- added TP62: H1-28, symbol Connector:TestPoint_Small
- added TP63: 3.3V_SYS (H2-27), symbol Connector:TestPoint_Small
- added TP64: 3.3V_SYS (H2-28), symbol Connector:TestPoint_Small
- added TP65: ~RESET~ (H1-29), symbol Connector:TestPoint_Small
- added TP66: H1-30, symbol Connector:TestPoint_Small
- added TP67: GND (H2-29), symbol Connector:TestPoint_Small
- added TP68: GND (H2-30), symbol Connector:TestPoint_Small
- added TP69: H1-31, symbol Connector:TestPoint_Small
- added TP7: -Z_SOLAR_PWR, symbol Connector:TestPoint_Small
- added TP70: 5V_USB (H1-32), symbol Connector:TestPoint_Small
- added TP71: AGND (H2-31), symbol Connector:TestPoint_Small
- added TP72: GND (H2-32), symbol Connector:TestPoint_Small
- added TP73: VCC_RF (H1-33), symbol Connector:TestPoint_Small
- added TP74: H1-34, symbol Connector:TestPoint_Small
- added TP75: H2-33, symbol Connector:TestPoint_Small
- added TP76: H2-34, symbol Connector:TestPoint_Small
- added TP77: H1-35, symbol Connector:TestPoint_Small
- added TP78: H1-36, symbol Connector:TestPoint_Small
- added TP79: H2-35, symbol Connector:TestPoint_Small
- added TP8: +X_SOLAR_PWR, symbol Connector:TestPoint_Small
- added TP80: H2-26, symbol Connector:TestPoint_Small
- added TP81: H1-37, symbol Connector:TestPoint_Small
- added TP82: H1-38, symbol Connector:TestPoint_Small
- added TP83: H2-37, symbol Connector:TestPoint_Small
- added TP84: H2-38, symbol Connector:TestPoint_Small
- added TP85: H1-39, symbol Connector:TestPoint_Small
- added TP86: H1-40, symbol Connector:TestPoint_Small
- added TP87: H2-39, symbol Connector:TestPoint_Small
- added TP88: H2-40, symbol Connector:TestPoint_Small
- added TP89: H1-41, symbol Connector:TestPoint_Small
- added TP9: H1-1, symbol Connector:TestPoint_Small
- added TP90: H1-42, symbol Connector:TestPoint_Small
- added TP91: H2-41, symbol Connector:TestPoint_Small
- added TP92: H2-42, symbol Connector:TestPoint_Small
- added TP93: H1-43, symbol Connector:TestPoint_Small
- added TP94: H1-44, symbol Connector:TestPoint_Small
- added TP95: H2-43, symbol Connector:TestPoint_Small
- added TP96: H2-44, symbol Connector:TestPoint_Small
- added TP97: VBATT+ (H2-45), symbol Connector:TestPoint_Small
- added TP98: VBATT+ (H1-46), symbol Connector:TestPoint_Small
- added TP99: USER_6 (H2-45), symbol Connector:TestPoint_Small
Connections:
- net labels added: 3.3V_SYS, 5V_DEBUG, 5V_SYS, USER_LED_1, USER_LED_2, USER_LED_3, USER_LED_4, USER_LED_5, USER_LED_6, USER_LED_7, USER_LED_8, USER_SW_1, USER_SW_1_RET, USER_SW_1_SEND, USER_SW_2, USER_SW_2_RET, USER_SW_2_SEND, USER_SW_3, USER_SW_3_RET, USER_SW_3_SEND, USER_SW_4, USER_SW_4_RET, USER_SW_4_SEND, VBATT, VBATT_RET, V_PLD, V_RF
- wire segments 120 -> 619
- no-connect marks 0 -> 7
Other:
- note added: "BACKPLANE CARD EDGE CONNECTOR"
- note added: "BREAKOUT CONNECTOR"
- note added: "BREAKOUT HEADERS"
- note added: "CONFIGURATION JUMPERS + SWITCHES"
- note added: "DISCRETE INDICATOR LEDs"
- note added: "DISCRETE USER LEDs"
- note added: "GND header to grab ground"
- note added: "GREEN PWR LEDs"
- note added: "PCB BOTTOM"
- note added: "PCB TOP"
- note added: "POWER DELIVERY + MEASUREMENT"
- note added: "POWER ENTRY MINI-NANA JACKS"
- note added: "RED SEP / RST LEDs"
- note added: "TEST POINTS"
- note added: "connecting this will send 5V debug to the backplane"
- note added: "displays the same data \nas on the LEDs on the backplane"
- note added: "user configurable switches, normally open"

Commit message: backplane-breakout-big
Parts:
- J1: footprint backplane-breakout-big:SAMTEC_LSH-030-01-X-D-A-TR -> backplane-breakout-big:SAMTEC_FTSH-130-04-L-DH; Manufacturer Part Number 1 LSH-030-01-X-D-A-TR -> FTSH-130-04-L-DH
- J2: footprint backplane-breakout-big:SAMTEC_LSH-030-01-X-D-A-TR -> backplane-breakout-big:SAMTEC_FTSH-130-04-L-DH_flipped; Manufacturer Part Number 1 LSH-030-01-X-D-A-TR -> FTSH-130-04-L-DH
- J20, J5: footprint (none) -> Connector_PinHeader_2.54mm:PinHeader_2x04_P2.54mm_Vertical_SMD
- J22, J23: value Conn_02x30_Odd_Even -> SSM-130-L-DV; footprint Connector_PinHeader_2.54mm:PinHeader_2x30_P2.54mm_Vertical -> backplane-breakout-big:SAMTEC_SSM-130-L-DV
- J24: value Conn_02x04_Odd_Even -> GND; footprint (none) -> Connector_PinHeader_2.54mm:PinHeader_2x04_P2.54mm_Vertical_SMD
- J3: footprint (none) -> Connector_PinHeader_2.54mm:PinHeader_1x02_P2.54mm_Vertical
- R1, R10, R11, R12, R13, R14, R15, R16, R17, R18, R19, R2, R20, R21, R22, R23, R24, R25, R26, R27, R28, R29, R3, R30, R31, R32, R33, R34, R35, R36, R37, R38, R39, R4, R5, R6, R7, R8, R9: footprint (none) -> Resistor_SMD:R_0603_1608Metric
- SW1, SW2, SW3, SW4, SW5, SW6, SW7, SW8, SW9: footprint backplane-breakout-big:SW_OS102011MS2QN1 -> backplane-breakout-big:JS102011SCQN
- TP1, TP10, TP100, TP101, TP102, TP103, TP104, TP105, TP106, TP107, TP108, TP109, TP11, TP110, TP111, TP112, TP113, TP114, TP115, TP116, TP117, TP118, TP119, TP12, TP120, TP13, TP14, TP15, TP16, TP17, TP18, TP19, TP2, TP20, TP21, TP22, TP23, TP24, TP25, TP26, TP28, TP29, TP3, TP30, TP31, TP32, TP33, TP34, TP35, TP36, TP37, TP38, TP39, TP4, TP40, TP41, TP42, TP43, TP44, TP45, TP46, TP47, TP48, TP49, TP5, TP50, TP51, TP52, TP53, TP54, TP55, TP56, TP57, TP58, TP59, TP6, TP60, TP61, TP62, TP63, TP64, TP65, TP66, TP67, TP68, TP69, TP7, TP70, TP71, TP72, TP73, TP74, TP75, TP76, TP77, TP78, TP79, TP8, TP81, TP82, TP83, TP84, TP85, TP86, TP87, TP88, TP89, TP9, TP90, TP91, TP92, TP93, TP94, TP95, TP96, TP97, TP98, TP99: footprint (none) -> backplane-breakout-big:Keystone_5027
- TP27: value H2-0 -> H2-9; footprint (none) -> backplane-breakout-big:Keystone_5027
- TP80: value H2-26 -> H2-36; footprint (none) -> backplane-breakout-big:Keystone_5027
Connections:
- wire segments 619 -> 617
Other:
- note removed: "displays the same data \nas on the LEDs on the backplane"
- moved on the sheet: J22, J23, J24
