File: backplane-boards/backplane-breakout-big/backplane-breaout-big.kicad_pcb (KiCad board)
At the start: 2 copper layers, 43 x 10 mm, 3 parts, among them J1 Breakout Connector, J2 Breakout Connector

Commit message: breakout-big
Parts:
- added C1: 0.1uF, Capacitor_SMD:C_0603_1608Metric, F.Cu at (200.6, 151.2)
- added C2: 0.1uF, Capacitor_SMD:C_0603_1608Metric, F.Cu at (208.6, 151.2)
- added D1: GREEN, LED_SMD:LED_0603_1608Metric_Castellated, F.Cu at (217.8, 101.1)
- added D10: GREEN, LED_SMD:LED_0603_1608Metric_Castellated, F.Cu at (213.3, 98.6)
- added D11: ORANGE, LED_SMD:LED_0603_1608Metric_Castellated, F.Cu at (217.8, 96.2)
- added D12: ORANGE, LED_SMD:LED_0603_1608Metric_Castellated, F.Cu at (213.3, 96.2)
- added D13: BLUE, LED_SMD:LED_0603_1608Metric_Castellated, F.Cu at (217.8, 110.9)
- added D14: BLUE, LED_SMD:LED_0603_1608Metric_Castellated, F.Cu at (238.9, 92.8)
- added D15: RED, LED_SMD:LED_0603_1608Metric_Castellated, F.Cu at (235.6, 96.4)
- added D16: RED, LED_SMD:LED_0603_1608Metric_Castellated, F.Cu at (231.2, 101.4)
- added D17: RED, LED_SMD:LED_0603_1608Metric_Castellated, F.Cu at (231.2, 98.9)
- added D18: RED, LED_SMD:LED_0603_1608Metric_Castellated, F.Cu at (231.2, 96.4)
- added D19: RED, LED_SMD:LED_0603_1608Metric_Castellated, F.Cu at (198.9, 131.8)
- added D2: GREEN, LED_SMD:LED_0603_1608Metric_Castellated, F.Cu at (213.3, 101.1)
- added D20: BLUE, LED_SMD:LED_0603_1608Metric_Castellated, F.Cu at (208.9, 103.6)
- added D21: RED, LED_SMD:LED_0603_1608Metric_Castellated, F.Cu at (208.9, 108.6)
- added D22: BLUE, LED_SMD:LED_0603_1608Metric_Castellated, F.Cu at (208.9, 106.1)
- added D23: RED, LED_SMD:LED_0603_1608Metric_Castellated, F.Cu at (213.3, 103.6)
- added D3: GREEN, LED_SMD:LED_0603_1608Metric_Castellated, F.Cu at (208.9, 101.1)
- added D4: ORANGE, LED_SMD:LED_0603_1608Metric_Castellated, F.Cu at (217.8, 98.6)
- added D5: GREEN, LED_SMD:LED_0603_1608Metric_Castellated, F.Cu at (230.0, 89.1)
- added D6: ORANGE, LED_SMD:LED_0603_1608Metric_Castellated, F.Cu at (208.9, 96.2)
- added D600_1: 156125M173000, backplane-breakout-big:156125M173000, F.Cu at (212.6, 144.3)
- added D600_2: 156125M173000, backplane-breakout-big:156125M173000, F.Cu at (207.1, 148.0)
- added D600_3: 156125M173000, backplane-breakout-big:156125M173000, F.Cu at (212.6, 140.6)
- added D600_4: 156125M173000, backplane-breakout-big:156125M173000, F.Cu at (201.5, 148.0)
- added D600_5: 156125M173000, backplane-breakout-big:156125M173000, F.Cu at (207.1, 144.3)
- added D600_6: 156125M173000, backplane-breakout-big:156125M173000, F.Cu at (201.5, 144.3)
- added D600_7: 156125M173000, backplane-breakout-big:156125M173000, F.Cu at (207.1, 140.6)
- added D600_8: 156125M173000, backplane-breakout-big:156125M173000, F.Cu at (201.5, 140.6)
- added D7: GREEN, LED_SMD:LED_0603_1608Metric_Castellated, F.Cu at (194.5, 131.8)
- added D8: GREEN, LED_SMD:LED_0603_1608Metric_Castellated, F.Cu at (208.9, 98.6)
- added D9: GREEN, LED_SMD:LED_0603_1608Metric_Castellated, F.Cu at (194.5, 134.2)
- added J10: -Z_SOLAR_RTN, backplane-breakout-big:Keystone_476, F.Cu at (217.2, 91.4)
- added J11: +Y_SOLAR_PWR, backplane-breakout-big:Keystone_476, F.Cu at (210.2, 77.3)
- added J12: +Y_SOLAR_RTN, backplane-breakout-big:Keystone_476, F.Cu at (252.4, 77.3)
- added J13: -X_SOLAR_PWR, backplane-breakout-big:Keystone_476, F.Cu at (210.2, 84.3)
- added J14: -X_SOLAR_RTN, backplane-breakout-big:Keystone_476, F.Cu at (217.2, 84.3)
- added J15: 3.3V_SYS, backplane-breakout-big:Keystone_476, F.Cu at (217.2, 77.3)
- added J16: +5V_SYS, backplane-breakout-big:Keystone_476, F.Cu at (224.3, 84.3)
- added J17: VCC_RF, backplane-breakout-big:Keystone_476, F.Cu at (231.3, 84.3)
- added J18: 5V_DEBUG, backplane-breakout-big:Keystone_476, F.Cu at (238.3, 84.3)
- added J19: GND, backplane-breakout-big:Keystone_476, F.Cu at (245.4, 84.3)
- added J200_1: HSEC8-160-01-S-DV-A-K-TR, backplane-breakout-big:HSEC8-160-01-S-DV-A-K-TR, F.Cu at (244.6, 56.8)
- added J21: AGND, backplane-breakout-big:Keystone_476, F.Cu at (224.3, 91.4)
- added J22: Conn_02x30_Odd_Even, Connector_PinHeader_2.54mm:PinHeader_2x30_P2.54mm_Vertical, F.Cu at (201.8, 54.5)
- added J23: Conn_02x30_Odd_Even, Connector_PinHeader_2.54mm:PinHeader_2x30_P2.54mm_Vertical, F.Cu at (194.6, 54.5)
- added J4: PACK+, backplane-breakout-big:Keystone_476, F.Cu at (224.3, 77.3)
- added J6: PACK-, backplane-breakout-big:Keystone_476, F.Cu at (231.3, 77.3)
- added J7: +X_SOLAR_PWR, backplane-breakout-big:Keystone_476, F.Cu at (238.3, 77.3)
- added J8: +X_SOLAR_RTN, backplane-breakout-big:Keystone_476, F.Cu at (245.4, 77.3)
- added J9: -Z_SOLAR_PWR, backplane-breakout-big:Keystone_476, F.Cu at (210.2, 91.4)
- added Q1: DMG1012UW-7, Package_TO_SOT_SMD:SOT-323_SC-70, F.Cu at (234.4, 89.7)
- added Q10: DMG1012UW-7, Package_TO_SOT_SMD:SOT-323_SC-70, F.Cu at (217.8, 114.0)
- added Q11: DMG1012UW-7, Package_TO_SOT_SMD:SOT-323_SC-70, F.Cu at (251.1, 82.7)
- added Q12: DMG1012UW-7, Package_TO_SOT_SMD:SOT-323_SC-70, F.Cu at (208.9, 121.3)
- added Q13: BSS84W-7-F, Package_TO_SOT_SMD:SOT-323_SC-70, F.Cu at (213.3, 117.6)
- added Q14: BSS84W-7-F, Package_TO_SOT_SMD:SOT-323_SC-70, F.Cu at (208.9, 117.6)
- added Q15: BSS84W-7-F, Package_TO_SOT_SMD:SOT-323_SC-70, F.Cu at (213.3, 114.0)
- added Q16: BSS84W-7-F, Package_TO_SOT_SMD:SOT-323_SC-70, F.Cu at (238.9, 89.7)
- added Q17: BSS84W-7-F, Package_TO_SOT_SMD:SOT-323_SC-70, F.Cu at (213.3, 106.7)
- added Q18: DMG1012UW-7, Package_TO_SOT_SMD:SOT-323_SC-70, F.Cu at (217.8, 107.8)
- added Q19: DMG1012UW-7, Package_TO_SOT_SMD:SOT-323_SC-70, F.Cu at (222.2, 107.7)
- added Q2: DMG1012UW-7, Package_TO_SOT_SMD:SOT-323_SC-70, F.Cu at (226.7, 96.7)
- added Q20: BSS84W-7-F, Package_TO_SOT_SMD:SOT-323_SC-70, F.Cu at (226.7, 104.0)
- added Q21: BSS84W-7-F, Package_TO_SOT_SMD:SOT-323_SC-70, F.Cu at (222.2, 104.0)
- added Q22: DMG1012UW-7, Package_TO_SOT_SMD:SOT-323_SC-70, F.Cu at (226.7, 100.4)
- added Q23: DMG1012UW-7, Package_TO_SOT_SMD:SOT-323_SC-70, F.Cu at (234.4, 93.3)
- added Q3: DMG1012UW-7, Package_TO_SOT_SMD:SOT-323_SC-70, F.Cu at (213.3, 110.3)
- added Q4: DMG1012UW-7, Package_TO_SOT_SMD:SOT-323_SC-70, F.Cu at (222.2, 100.4)
- added Q5: DMG1012UW-7, Package_TO_SOT_SMD:SOT-323_SC-70, F.Cu at (217.8, 104.2)
- added Q6: DMG1012UW-7, Package_TO_SOT_SMD:SOT-323_SC-70, F.Cu at (208.9, 111.7)
- added Q7: DMG1012UW-7, Package_TO_SOT_SMD:SOT-323_SC-70, F.Cu at (230.0, 92.2)
- added Q8: DMG1012UW-7, Package_TO_SOT_SMD:SOT-323_SC-70, F.Cu at (222.2, 111.3)
- added Q9: DMG1012UW-7, Package_TO_SOT_SMD:SOT-323_SC-70, F.Cu at (222.2, 96.7)
- added R40: 50.1k, Resistor_SMD:R_0603_1608Metric, F.Cu at (211.7, 147.4)
- added R41: 50.1k, Resistor_SMD:R_0603_1608Metric, F.Cu at (204.6, 151.2)
- added SW1: SEP1, backplane-breakout-big:SW_OS102011MS2QN1, F.Cu at (225.5, 65.0)
- added SW2: SEP2, backplane-breakout-big:SW_OS102011MS2QN1, F.Cu at (237.8, 65.0)
- added SW3: SEP3, backplane-breakout-big:SW_OS102011MS2QN1, F.Cu at (225.5, 70.9)
- added SW4: SEP4, backplane-breakout-big:SW_OS102011MS2QN1, F.Cu at (237.8, 70.9)
- added SW5: RBF, backplane-breakout-big:SW_OS102011MS2QN1, F.Cu at (250.2, 70.9)
- added SW6: USER_SW_1, backplane-breakout-big:SW_OS102011MS2QN1, F.Cu at (213.2, 65.0)
- added SW7: USER_SW_2, backplane-breakout-big:SW_OS102011MS2QN1, F.Cu at (213.2, 70.9)
- added SW8: USER_SW_3, backplane-breakout-big:SW_OS102011MS2QN1, F.Cu at (262.5, 65.0)
- added SW9: USER_SW_4, backplane-breakout-big:SW_OS102011MS2QN1, F.Cu at (250.2, 65.0)
- added U1: TLC59282, Package_DFN_QFN:VQFN-24-1EP_4x4mm_P0.5mm_EP2.45x2.45mm, F.Cu at (195.4, 141.9)
- added U2: TLC59282, Package_DFN_QFN:VQFN-24-1EP_4x4mm_P0.5mm_EP2.45x2.45mm, F.Cu at (195.4, 148.2)
- J1, J2: footprint backplane-rbf:SAMTEC_LSH-030-01-X-D-A-TR -> backplane-breakout-big:SAMTEC_LSH-030-01-X-D-A-TR
Connections:
- J1 pad 59: /H2-25 -> 5V_SYS
- J1 pad 60: /H2-26 -> 5V_SYS
- J2 pad 12: /GND -> EP
- J2 pad 13: /H1-33 -> V_RF
- J2 pad 3: /H2-27 -> 3.3V_SYS
- J2 pad 39: /H2-45 -> VBATT
- J2 pad 4: /H2-28 -> 3.3V_SYS
- J2 pad 40: /H2-46 -> VBATT
- J2 pad 43: /GND -> EP
- J2 pad 44: /GND -> EP
- J2 pad 47: /H2-49 -> VBATT_RET
- J2 pad 48: /H2-50 -> VBATT_RET
- J2 pad 7: /GND -> EP
- J2 pad 8: /GND -> EP
Other:
- board text removed: "RBF"
- board text removed: "REMOVE BEFORE FLIGHT"
- board text removed: "please"

Commit message: backplane-breakout-big
Parts:
- removed C1, C2: 0.1uF, Capacitor_SMD:C_0603_1608Metric
- removed D600_1, D600_2, D600_3, D600_4, D600_5, D600_6, D600_7, D600_8: 156125M173000, backplane-breakout-big:156125M173000
- removed NT1: Net-Tie_2, backplane-rbf:NetTie-2_SMD_Pad0.25mm
- removed R40, R41: 50.1k, Resistor_SMD:R_0603_1608Metric
- removed U1, U2: TLC59282, Package_DFN_QFN:VQFN-24-1EP_4x4mm_P0.5mm_EP2.45x2.45mm
- added J20: Conn_02x04_Odd_Even, Connector_PinHeader_2.54mm:PinHeader_2x04_P2.54mm_Vertical_SMD, F.Cu at (123.0, 167.6)
- added J24: GND, Connector_PinHeader_2.54mm:PinHeader_2x04_P2.54mm_Vertical_SMD, F.Cu at (99.5, 167.6)
- added J3: DEBUG POWER SEND JUMPER, Connector_PinHeader_2.54mm:PinHeader_1x02_P2.54mm_Vertical, F.Cu at (69.5, 73.5)
- added J5: Conn_01x08, Connector_PinHeader_2.54mm:PinHeader_2x04_P2.54mm_Vertical_SMD, F.Cu at (239.4, 144.8)
- added R1: 1k, Resistor_SMD:R_0603_1608Metric, F.Cu at (143.3, 171.4)
- added R10: 10k, Resistor_SMD:R_0603_1608Metric, F.Cu at (218.8, 167.0)
- added R11: 10k, Resistor_SMD:R_0603_1608Metric, F.Cu at (157.9, 167.0)
- added R12: 10k, Resistor_SMD:R_0603_1608Metric, F.Cu at (223.9, 167.0)
- added R13: 1k, Resistor_SMD:R_0603_1608Metric, F.Cu at (163.6, 171.4)
- added R14: 1k, Resistor_SMD:R_0603_1608Metric, F.Cu at (168.7, 171.4)
- added R15: 1k, Resistor_SMD:R_0603_1608Metric, F.Cu at (173.8, 171.4)
- added R16: 1k, Resistor_SMD:R_0603_1608Metric, F.Cu at (178.8, 171.4)
- added R17: 1k, Resistor_SMD:R_0603_1608Metric, F.Cu at (229.6, 171.4)
- added R18: 1k, Resistor_SMD:R_0603_1608Metric, F.Cu at (234.7, 171.4)
- added R19: 10k, Resistor_SMD:R_0603_1608Metric, F.Cu at (163.0, 167.0)
- added R2: 1k, Resistor_SMD:R_0603_1608Metric, F.Cu at (148.4, 171.4)
- added R20: 10k, Resistor_SMD:R_0603_1608Metric, F.Cu at (168.0, 167.0)
- added R21: 10k, Resistor_SMD:R_0603_1608Metric, F.Cu at (173.1, 167.0)
- added R22: 10k, Resistor_SMD:R_0603_1608Metric, F.Cu at (178.2, 167.0)
- added R23: 10k, Resistor_SMD:R_0603_1608Metric, F.Cu at (229.0, 167.0)
- added R24: 10k, Resistor_SMD:R_0603_1608Metric, F.Cu at (234.1, 167.0)
- added R25: 1k, Resistor_SMD:R_0603_1608Metric, F.Cu at (239.8, 171.4)
- added R26: 1k, Resistor_SMD:R_0603_1608Metric, F.Cu at (244.9, 171.4)
- added R27: 1k, Resistor_SMD:R_0603_1608Metric, F.Cu at (183.9, 171.4)
- added R28: 1k, Resistor_SMD:R_0603_1608Metric, F.Cu at (189.0, 171.4)
- added R29: 1k, Resistor_SMD:R_0603_1608Metric, F.Cu at (194.1, 171.4)
- added R3: 1k, Resistor_SMD:R_0603_1608Metric, F.Cu at (153.4, 171.4)
- added R30: 1k, Resistor_SMD:R_0603_1608Metric, F.Cu at (199.2, 171.4)
- added R31: 1k, Resistor_SMD:R_0603_1608Metric, F.Cu at (204.2, 171.4)
- added R32: 10k, Resistor_SMD:R_0603_1608Metric, F.Cu at (239.2, 167.0)
- added R33: 10k, Resistor_SMD:R_0603_1608Metric, F.Cu at (244.2, 167.0)
- added R34: 1k, Resistor_SMD:R_0603_1608Metric, F.Cu at (250.0, 171.4)
- added R35: 1k, Resistor_SMD:R_0603_1608Metric, F.Cu at (209.3, 171.4)
- added R36: 1k, Resistor_SMD:R_0603_1608Metric, F.Cu at (255.0, 171.4)
- added R37: 1k, Resistor_SMD:R_0603_1608Metric, F.Cu at (214.4, 171.4)
- added R38: 10k, Resistor_SMD:R_0603_1608Metric, F.Cu at (249.3, 167.0)
- added R39: 10k, Resistor_SMD:R_0603_1608Metric, F.Cu at (254.4, 167.0)
- added R4: 1k, Resistor_SMD:R_0603_1608Metric, F.Cu at (219.5, 171.4)
- added R5: 1k, Resistor_SMD:R_0603_1608Metric, F.Cu at (158.5, 171.4)
- added R6: 1k, Resistor_SMD:R_0603_1608Metric, F.Cu at (224.6, 171.4)
- added R7: 10k, Resistor_SMD:R_0603_1608Metric, F.Cu at (142.6, 167.0)
- added R8: 10k, Resistor_SMD:R_0603_1608Metric, F.Cu at (147.7, 167.0)
- added R9: 10k, Resistor_SMD:R_0603_1608Metric, F.Cu at (152.8, 167.0)
- added TP1: SEP1, backplane-breakout-big:Keystone_5027, F.Cu at (145.4, 85.1)
- added TP10: H1-2, backplane-breakout-big:Keystone_5027, F.Cu at (145.4, 104.1)
- added TP100: H2-46, backplane-breakout-big:Keystone_5027, F.Cu at (240.7, 88.9)
- added TP101: SELF_TEST (H1-47), backplane-breakout-big:Keystone_5027, F.Cu at (183.5, 138.4)
- added TP102: USER_1 (H1-48), backplane-breakout-big:Keystone_5027, F.Cu at (183.5, 142.2)
- added TP103: GND (H2-47), backplane-breakout-big:Keystone_5027, F.Cu at (240.7, 92.5)
- added TP104: GND (H2-48), backplane-breakout-big:Keystone_5027, F.Cu at (240.7, 96.3)
- added TP105: USER_2 (H1-49), backplane-breakout-big:Keystone_5027, F.Cu at (183.5, 146.1)
- added TP106: USER_3 (H1-50), backplane-breakout-big:Keystone_5027, F.Cu at (183.5, 149.9)
- added TP107: VBATT- (H2-49), backplane-breakout-big:Keystone_5027, F.Cu at (240.7, 100.1)
- added TP108: VBATT- (H2-50), backplane-breakout-big:Keystone_5027, F.Cu at (240.7, 103.9)
- added TP109: USER_4 (H1-51), backplane-breakout-big:Keystone_5027, F.Cu at (202.6, 62.2)
- added TP11: H2-1, backplane-breakout-big:Keystone_5027, F.Cu at (202.6, 100.3)
- added TP110: USER_5 (H1-52), backplane-breakout-big:Keystone_5027, F.Cu at (202.6, 66.0)
- added TP111: USER_10 (H2-51), backplane-breakout-big:Keystone_5027, F.Cu at (240.7, 108.0)
- added TP112: USER_11 (H2-52), backplane-breakout-big:Keystone_5027, F.Cu at (240.7, 111.8)
- added TP113: +Y_SOLAR_TLE, backplane-breakout-big:Keystone_5027, F.Cu at (202.6, 69.8)
- added TP114: -X_SOLAR_TLE, backplane-breakout-big:Keystone_5027, F.Cu at (202.6, 73.7)
- added TP115: +Y_SOLAR_RTN, backplane-breakout-big:Keystone_5027, F.Cu at (240.7, 115.6)
- added TP116: -X_SOLAR_RTN, backplane-breakout-big:Keystone_5027, F.Cu at (240.7, 119.4)
- added TP117: +Y_SOLAR_PWR, backplane-breakout-big:Keystone_5027, F.Cu at (202.6, 77.5)
- added TP118: -X_SOLAR_PWR, backplane-breakout-big:Keystone_5027, F.Cu at (202.6, 81.3)
- added TP119: SEP3, backplane-breakout-big:Keystone_5027, F.Cu at (240.7, 123.2)
- added TP12: H2-2, backplane-breakout-big:Keystone_5027, F.Cu at (202.6, 104.1)
- added TP120: SEP4, backplane-breakout-big:Keystone_5027, F.Cu at (240.7, 127.0)
- added TP13: H1-3, backplane-breakout-big:Keystone_5027, F.Cu at (145.4, 108.0)
- added TP14: H1-4, backplane-breakout-big:Keystone_5027, F.Cu at (145.4, 111.8)
- added TP15: H2-3, backplane-breakout-big:Keystone_5027, F.Cu at (202.6, 108.0)
- added TP16: H2-4, backplane-breakout-big:Keystone_5027, F.Cu at (202.6, 111.8)
- added TP17: H1-5, backplane-breakout-big:Keystone_5027, F.Cu at (145.4, 115.6)
- added TP18: H1-6, backplane-breakout-big:Keystone_5027, F.Cu at (145.4, 119.4)
- added TP19: H2-5, backplane-breakout-big:Keystone_5027, F.Cu at (202.6, 115.6)
- added TP2: SEP2, backplane-breakout-big:Keystone_5027, F.Cu at (145.4, 88.9)
- added TP20: H2-6, backplane-breakout-big:Keystone_5027, F.Cu at (202.6, 119.4)
- added TP21: H1-7, backplane-breakout-big:Keystone_5027, F.Cu at (145.4, 123.2)
- added TP22: H1-8, backplane-breakout-big:Keystone_5027, F.Cu at (145.4, 127.0)
- added TP23: H2-7, backplane-breakout-big:Keystone_5027, F.Cu at (202.6, 123.2)
- added TP24: H2-8, backplane-breakout-big:Keystone_5027, F.Cu at (202.6, 127.0)
- added TP25: H1-9, backplane-breakout-big:Keystone_5027, F.Cu at (145.4, 130.8)
- added TP26: H1-10, backplane-breakout-big:Keystone_5027, F.Cu at (145.4, 134.6)
- added TP27: H2-9, backplane-breakout-big:Keystone_5027, F.Cu at (202.6, 130.8)
- added TP28: H2-10, backplane-breakout-big:Keystone_5027, F.Cu at (202.6, 134.6)
- added TP29: H1-11, backplane-breakout-big:Keystone_5027, F.Cu at (145.4, 138.4)
- added TP3: -Z_SOLAR_TLE, backplane-breakout-big:Keystone_5027, F.Cu at (202.6, 85.1)
- added TP30: H1-12, backplane-breakout-big:Keystone_5027, F.Cu at (145.4, 142.2)
- added TP31: H2-11, backplane-breakout-big:Keystone_5027, F.Cu at (202.6, 138.4)
- added TP32: H2-12, backplane-breakout-big:Keystone_5027, F.Cu at (202.6, 142.2)
- added TP33: H1-13, backplane-breakout-big:Keystone_5027, F.Cu at (145.4, 146.1)
- added TP34: H1-14, backplane-breakout-big:Keystone_5027, F.Cu at (145.4, 149.9)
- added TP35: H2-13, backplane-breakout-big:Keystone_5027, F.Cu at (202.6, 146.1)
- added TP36: H2-14, backplane-breakout-big:Keystone_5027, F.Cu at (202.6, 149.9)
- added TP37: RBF (H1-15), backplane-breakout-big:Keystone_5027, F.Cu at (164.5, 85.1)
- added TP38: H1-16, backplane-breakout-big:Keystone_5027, F.Cu at (164.5, 88.9)
- added TP39: H2-15, backplane-breakout-big:Keystone_5027, F.Cu at (221.6, 62.2)
- added TP4: +X_SOLAR_TLE, backplane-breakout-big:Keystone_5027, F.Cu at (202.6, 88.9)
- added TP40: H2-16, backplane-breakout-big:Keystone_5027, F.Cu at (221.6, 66.0)
- added TP41: H1-17, backplane-breakout-big:Keystone_5027, F.Cu at (164.5, 92.7)
- added TP42: H1-18, backplane-breakout-big:Keystone_5027, F.Cu at (164.5, 96.5)
- added TP43: H2-17, backplane-breakout-big:Keystone_5027, F.Cu at (221.6, 69.8)
- added TP44: H2-18, backplane-breakout-big:Keystone_5027, F.Cu at (221.6, 73.7)
- added TP45: H1-19, backplane-breakout-big:Keystone_5027, F.Cu at (164.5, 100.3)
- added TP46: H1-20, backplane-breakout-big:Keystone_5027, F.Cu at (164.5, 104.1)
- added TP47: H2-19, backplane-breakout-big:Keystone_5027, F.Cu at (221.6, 77.5)
- added TP48: H2-20, backplane-breakout-big:Keystone_5027, F.Cu at (221.6, 81.3)
- added TP49: H1-21, backplane-breakout-big:Keystone_5027, F.Cu at (164.5, 108.0)
- added TP5: -Z_SOLAR_RTN, backplane-breakout-big:Keystone_5027, F.Cu at (145.4, 92.7)
- added TP50: H1-22, backplane-breakout-big:Keystone_5027, F.Cu at (164.5, 111.8)
- added TP51: H2-21, backplane-breakout-big:Keystone_5027, F.Cu at (221.6, 85.1)
- added TP52: H2-22, backplane-breakout-big:Keystone_5027, F.Cu at (221.6, 88.9)
- added TP53: H1-23, backplane-breakout-big:Keystone_5027, F.Cu at (164.5, 115.6)
- added TP54: H1-24, backplane-breakout-big:Keystone_5027, F.Cu at (164.5, 119.4)
- added TP55: H2-23, backplane-breakout-big:Keystone_5027, F.Cu at (221.6, 92.7)
- added TP56: H2-24, backplane-breakout-big:Keystone_5027, F.Cu at (221.6, 96.5)
- added TP57: H1-25, backplane-breakout-big:Keystone_5027, F.Cu at (164.5, 123.2)
- added TP58: H1-26, backplane-breakout-big:Keystone_5027, F.Cu at (164.5, 127.0)
- added TP59: 5V_SYS (H2-25), backplane-breakout-big:Keystone_5027, F.Cu at (221.6, 100.3)
- added TP6: +X_SOLAR_RTN, backplane-breakout-big:Keystone_5027, F.Cu at (145.4, 96.5)
- added TP60: 5V_SYS (H2-26), backplane-breakout-big:Keystone_5027, F.Cu at (221.6, 104.1)
- added TP61: H1-27, backplane-breakout-big:Keystone_5027, F.Cu at (164.5, 130.8)
- added TP62: H1-28, backplane-breakout-big:Keystone_5027, F.Cu at (164.5, 134.6)
- added TP63: 3.3V_SYS (H2-27), backplane-breakout-big:Keystone_5027, F.Cu at (221.6, 108.0)
- added TP64: 3.3V_SYS (H2-28), backplane-breakout-big:Keystone_5027, F.Cu at (221.6, 111.8)
- added TP65: ~RESET~ (H1-29), backplane-breakout-big:Keystone_5027, F.Cu at (164.5, 138.4)
- added TP66: H1-30, backplane-breakout-big:Keystone_5027, F.Cu at (164.5, 142.2)
- added TP67: GND (H2-29), backplane-breakout-big:Keystone_5027, F.Cu at (221.6, 115.6)
- added TP68: GND (H2-30), backplane-breakout-big:Keystone_5027, F.Cu at (221.6, 119.4)
- added TP69: H1-31, backplane-breakout-big:Keystone_5027, F.Cu at (164.5, 146.1)
- added TP7: -Z_SOLAR_PWR, backplane-breakout-big:Keystone_5027, F.Cu at (202.6, 92.7)
- added TP70: 5V_USB (H1-32), backplane-breakout-big:Keystone_5027, F.Cu at (164.5, 149.9)
- added TP71: AGND (H2-31), backplane-breakout-big:Keystone_5027, F.Cu at (221.6, 123.2)
- added TP72: GND (H2-32), backplane-breakout-big:Keystone_5027, F.Cu at (221.6, 127.0)
- added TP73: VCC_RF (H1-33), backplane-breakout-big:Keystone_5027, F.Cu at (183.5, 85.1)
- added TP74: H1-34, backplane-breakout-big:Keystone_5027, F.Cu at (183.5, 88.9)
- added TP75: H2-33, backplane-breakout-big:Keystone_5027, F.Cu at (221.6, 130.8)
- added TP76: H2-34, backplane-breakout-big:Keystone_5027, F.Cu at (221.6, 134.6)
- added TP77: H1-35, backplane-breakout-big:Keystone_5027, F.Cu at (183.5, 92.7)
- added TP78: H1-36, backplane-breakout-big:Keystone_5027, F.Cu at (183.5, 96.5)
- added TP79: H2-35, backplane-breakout-big:Keystone_5027, F.Cu at (221.6, 138.4)
- added TP8: +X_SOLAR_PWR, backplane-breakout-big:Keystone_5027, F.Cu at (202.6, 96.5)
- added TP80: H2-36, backplane-breakout-big:Keystone_5027, F.Cu at (221.6, 142.2)
- added TP81: H1-37, backplane-breakout-big:Keystone_5027, F.Cu at (183.5, 100.3)
- added TP82: H1-38, backplane-breakout-big:Keystone_5027, F.Cu at (183.5, 104.1)
- added TP83: H2-37, backplane-breakout-big:Keystone_5027, F.Cu at (221.6, 146.1)
- added TP84: H2-38, backplane-breakout-big:Keystone_5027, F.Cu at (221.6, 149.9)
- added TP85: H1-39, backplane-breakout-big:Keystone_5027, F.Cu at (183.5, 108.0)
- added TP86: H1-40, backplane-breakout-big:Keystone_5027, F.Cu at (183.5, 111.8)
- added TP87: H2-39, backplane-breakout-big:Keystone_5027, F.Cu at (240.7, 62.2)
- added TP88: H2-40, backplane-breakout-big:Keystone_5027, F.Cu at (240.7, 66.0)
- added TP89: H1-41, backplane-breakout-big:Keystone_5027, F.Cu at (183.5, 115.6)
- added TP9: H1-1, backplane-breakout-big:Keystone_5027, F.Cu at (145.4, 100.3)
- added TP90: H1-42, backplane-breakout-big:Keystone_5027, F.Cu at (183.5, 119.4)
- added TP91: H2-41, backplane-breakout-big:Keystone_5027, F.Cu at (240.7, 69.8)
- added TP92: H2-42, backplane-breakout-big:Keystone_5027, F.Cu at (240.7, 73.7)
- added TP93: H1-43, backplane-breakout-big:Keystone_5027, F.Cu at (183.5, 123.2)
- added TP94: H1-44, backplane-breakout-big:Keystone_5027, F.Cu at (183.5, 127.0)
- added TP95: H2-43, backplane-breakout-big:Keystone_5027, F.Cu at (240.7, 77.5)
- added TP96: H2-44, backplane-breakout-big:Keystone_5027, F.Cu at (240.7, 81.3)
- added TP97: VBATT+ (H2-45), backplane-breakout-big:Keystone_5027, F.Cu at (183.5, 130.8)
- added TP98: VBATT+ (H1-46), backplane-breakout-big:Keystone_5027, F.Cu at (183.5, 134.6)
- added TP99: USER_6 (H2-45), backplane-breakout-big:Keystone_5027, F.Cu at (240.7, 85.1)
- J1: footprint backplane-breakout-big:SAMTEC_LSH-030-01-X-D-A-TR -> backplane-breakout-big:SAMTEC_FTSH-130-04-L-DH; moved to F.Cu
- J2: footprint backplane-breakout-big:SAMTEC_LSH-030-01-X-D-A-TR -> backplane-breakout-big:SAMTEC_FTSH-130-04-L-DH_flipped
- J22, J23: value Conn_02x30_Odd_Even -> SSM-130-L-DV; footprint Connector_PinHeader_2.54mm:PinHeader_2x30_P2.54mm_Vertical -> backplane-breakout-big:SAMTEC_SSM-130-L-DV
- SW1, SW2, SW3, SW4, SW5, SW6, SW7, SW8, SW9: footprint backplane-breakout-big:SW_OS102011MS2QN1 -> backplane-breakout-big:JS102011SCQN
- moved J12 185.8 mm to (72.2, 122.4), turned to 270 degrees
- moved J19 184.0 mm to (72.2, 146.5)
- moved J17 182.7 mm to (59.5, 146.5)
- moved J15 182.3 mm to (59.5, 168.8)
- moved J7 181.8 mm to (59.5, 109.7), turned to 90 degrees
- moved J16 180.5 mm to (59.5, 158.0)
- moved J18 179.3 mm to (59.5, 72.2)
- moved J8 176.2 mm to (72.2, 109.7), turned to 270 degrees
- moved J4 174.6 mm to (59.5, 135.1), turned to 90 degrees
- moved J21 165.8 mm to (72.2, 157.3)
- moved J6 159.3 mm to (72.2, 84.3), turned to 270 degrees
- moved J13 155.5 mm to (59.5, 122.4), turned to 90 degrees
- moved J11 152.0 mm to (59.5, 97.0), turned to 90 degrees
- moved J10 151.5 mm to (72.2, 135.1)
- moved J9 150.9 mm to (59.5, 84.3), turned to 90 degrees
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Connections:
- D15 pad 1: EP -> GND
- D16 pad 1: EP -> GND
- D17 pad 1: EP -> GND
- D18 pad 1: EP -> GND
- D19 pad 1: EP -> GND
- D21 pad 1: EP -> GND
- D23 pad 1: EP -> GND
- J1 pad 10: /H1-2 -> /H1-6
- J1 pad 11: /H2-1 -> /H1-7
- J1 pad 12: /H2-2 -> /H1-8
- J1 pad 13: /H1-3 -> /H1-9
- J1 pad 14: /H1-4 -> /H1-10
- J1 pad 15: /H2-3 -> /H1-11
- J1 pad 16: /H2-4 -> /H1-12
- J1 pad 17: /H1-5 -> /H1-13
- J1 pad 18: /H1-6 -> /H1-14
- J1 pad 19: /H2-5 -> /RBF
- J1 pad 20: /H2-6 -> /H1-16
- J1 pad 21: /H1-7 -> /H1-17
- J1 pad 22: /H1-8 -> /H1-18
- J1 pad 23: /H2-7 -> /H1-19
- J1 pad 24: /H2-8 -> /H1-20
- J1 pad 25: /H1-9 -> /H1-21
- J1 pad 26: /H1-10 -> /H1-22
- J1 pad 27: /H2-9 -> /H1-23
- J1 pad 28: /H2-10 -> /H1-24
- J1 pad 29: /H1-11 -> /H1-25
- J1 pad 3: /-Z_SOLAR_TLE -> /-Z_SOLAR_RTN
- J1 pad 30: /H1-12 -> /H1-26
- J1 pad 31: /H2-11 -> /H1-27
- J1 pad 32: /H2-12 -> /H1-28
- J1 pad 33: /H1-13 -> /BUS_RESET
- J1 pad 34: /H1-14 -> /H1-30
- J1 pad 35: /H2-13 -> /H1-31
- J1 pad 36: /H2-14 -> /5V_USB
- J1 pad 37: /RBF -> V_RF
- J1 pad 38: /H1-16 -> /H1-34
- J1 pad 39: /H2-15 -> /H1-35
- J1 pad 4: /+X_SOLAR_TLE -> /+X_SOLAR_RTN
- J1 pad 40: /H2-16 -> /H1-36
- J1 pad 41: /H1-17 -> /H1-37
- J1 pad 42: /H1-18 -> /H1-38
- J1 pad 43: /H2-17 -> /H1-39
- J1 pad 44: /H2-18 -> /H1-40
- J1 pad 45: /H1-19 -> /H1-41
- J1 pad 46: /H1-20 -> /H1-42
- J1 pad 47: /H2-19 -> /H1-43
- J1 pad 48: /H2-20 -> /H1-44
- J1 pad 49: /H1-21 -> /H1-45
- J1 pad 5: /-Z_SOLAR_RTN -> /H1-1
- J1 pad 50: /H1-22 -> /H1-46
- J1 pad 51: /H2-21 -> /SELF_TEST
- J1 pad 52: /H2-22 -> /USER_1
- J1 pad 53: /H1-23 -> /USER_2
- J1 pad 54: /H1-24 -> /USER_3
- J1 pad 55: /H2-23 -> /H1-51
- J1 pad 56: /H2-24 -> /H1-52
- J1 pad 57: /H1-25 -> /+Y_SOLAR_TLE
- J1 pad 58: /H1-26 -> /-X_SOLAR_TLE
- J1 pad 59: 5V_SYS -> /+Y_SOLAR_PWR
- J1 pad 6: /+X_SOLAR_RTN -> /H1-2
- J1 pad 60: 5V_SYS -> /-X_SOLAR_PWR
- J1 pad 7: /-Z_SOLAR_PWR -> /H1-3
- J1 pad 8: /+X_SOLAR_PWR -> /H1-4
- J1 pad 9: /H1-1 -> /H1-5
- J19 pad 1: EP -> GND
- J2 pad 1: /H1-27 -> /-Z_SOLAR_TLE
- J2 pad 10: /5V_USB -> /H2-6
- J2 pad 11: /AGND -> /H2-7
- J2 pad 12: EP -> /H2-8
- J2 pad 13: V_RF -> /H2-9
- J2 pad 14: /H1-34 -> /H2-10
- J2 pad 15: /H2-33 -> /H2-11
- J2 pad 16: /H2-34 -> /H2-12
- J2 pad 17: /H1-35 -> /H2-13
- J2 pad 18: /H1-36 -> /H2-14
- J2 pad 19: /H2-35 -> /H2-15
- J2 pad 2: /H1-28 -> /+X_SOLAR_TLE
- J2 pad 20: /H2-36 -> /H2-16
- J2 pad 21: /H1-37 -> /H2-17
- J2 pad 22: /H1-38 -> /H2-18
- J2 pad 23: /H2-37 -> /H2-19
- J2 pad 24: /H2-38 -> /H2-20
- J2 pad 25: /H1-39 -> /H2-21
- J2 pad 26: /H1-40 -> /H2-22
- J2 pad 27: /H2-39 -> /H2-23
- J2 pad 28: /H2-40 -> /H2-24
- J2 pad 29: /H1-41 -> 5V_SYS
- J2 pad 3: 3.3V_SYS -> /-Z_SOLAR_PWR
- J2 pad 30: /H1-42 -> 5V_SYS
- J2 pad 31: /H2-41 -> 3.3V_SYS
- J2 pad 32: /H2-42 -> 3.3V_SYS
- J2 pad 33: /H1-43 -> GND
- J2 pad 34: /H1-44 -> GND
- J2 pad 35: /H2-43 -> /AGND
- J2 pad 36: /H2-44 -> GND
- J2 pad 37: /H1-45 -> /H2-33
- J2 pad 38: /H1-46 -> /H2-34
- J2 pad 39: VBATT -> /H2-35
- J2 pad 4: 3.3V_SYS -> /+X_SOLAR_PWR
- J2 pad 40: VBATT -> /H2-36
- J2 pad 41: /SELF_TEST -> /H2-37
- J2 pad 42: /USER_1 -> /H2-38
- J2 pad 43: EP -> /H2-39
- J2 pad 44: EP -> /H2-40
- J2 pad 45: /USER_2 -> /H2-41
- J2 pad 46: /USER_3 -> /H2-42
- J2 pad 47: VBATT_RET -> /H2-43
- J2 pad 48: VBATT_RET -> /H2-44
- J2 pad 49: /H1-51 -> VBATT
- J2 pad 5: /BUS_RESET -> /H2-1
- J2 pad 50: /H1-52 -> VBATT
- J2 pad 51: /H2-51 -> GND
- J2 pad 52: /H2-52 -> GND
- J2 pad 53: /+Y_SOLAR_TLE -> VBATT_RET
- J2 pad 54: /-X_SOLAR_TLE -> VBATT_RET
- J2 pad 55: /+Y_SOLAR_RTN -> /H2-51
- J2 pad 56: /-X_SOLAR_RTN -> /H2-52
- J2 pad 57: /+Y_SOLAR_PWR -> /+Y_SOLAR_RTN
- J2 pad 58: /-X_SOLAR_PWR -> /-X_SOLAR_RTN
- J2 pad 6: /H1-30 -> /H2-2
- J2 pad 7: EP -> /H2-3
- J2 pad 8: EP -> /H2-4
- J2 pad 9: /H1-31 -> /H2-5
- J200_1 pad 103: EP -> GND
- J200_1 pad 104: EP -> GND
- J200_1 pad 67: EP -> GND
- J200_1 pad 68: EP -> GND
- J200_1 pad 72: EP -> GND
- J22 pad 10: /H1-2 -> /H1-6
- J22 pad 11: /H2-1 -> /H1-7
- J22 pad 12: /H2-2 -> /H1-8
- J22 pad 13: /H1-3 -> /H1-9
- J22 pad 14: /H1-4 -> /H1-10
- J22 pad 15: /H2-3 -> /H1-11
- J22 pad 16: /H2-4 -> /H1-12
- J22 pad 17: /H1-5 -> /H1-13
- J22 pad 18: /H1-6 -> /H1-14
- J22 pad 19: /H2-5 -> /RBF
- J22 pad 20: /H2-6 -> /H1-16
- J22 pad 21: /H1-7 -> /H1-17
- J22 pad 22: /H1-8 -> /H1-18
- J22 pad 23: /H2-7 -> /H1-19
- J22 pad 24: /H2-8 -> /H1-20
- J22 pad 25: /H1-9 -> /H1-21
- J22 pad 26: /H1-10 -> /H1-22
- J22 pad 27: /H2-9 -> /H1-23
- J22 pad 28: /H2-10 -> /H1-24
- J22 pad 29: /H1-11 -> /H1-25
- J22 pad 3: /-Z_SOLAR_TLE -> /-Z_SOLAR_RTN
- J22 pad 30: /H1-12 -> /H1-26
- J22 pad 31: /H2-11 -> /H1-27
- J22 pad 32: /H2-12 -> /H1-28
- J22 pad 33: /H1-13 -> /BUS_RESET
- J22 pad 34: /H1-14 -> /H1-30
- J22 pad 35: /H2-13 -> /H1-31
- J22 pad 36: /H2-14 -> /5V_USB
- J22 pad 37: /RBF -> V_RF
- J22 pad 38: /H1-16 -> /H1-34
- J22 pad 39: /H2-15 -> /H1-35
- J22 pad 4: /+X_SOLAR_TLE -> /+X_SOLAR_RTN
- J22 pad 40: /H2-16 -> /H1-36
- J22 pad 41: /H1-17 -> /H1-37
- J22 pad 42: /H1-18 -> /H1-38
- J22 pad 43: /H2-17 -> /H1-39
- J22 pad 44: /H2-18 -> /H1-40
- J22 pad 45: /H1-19 -> /H1-41
- J22 pad 46: /H1-20 -> /H1-42
- J22 pad 47: /H2-19 -> /H1-43
- J22 pad 48: /H2-20 -> /H1-44
- J22 pad 49: /H1-21 -> /H1-45
- J22 pad 5: /-Z_SOLAR_RTN -> /H1-1
- J22 pad 50: /H1-22 -> /H1-46
- J22 pad 51: /H2-21 -> /SELF_TEST
- J22 pad 52: /H2-22 -> /USER_1
- J22 pad 53: /H1-23 -> /USER_2
- J22 pad 54: /H1-24 -> /USER_3
- J22 pad 55: /H2-23 -> /H1-51
- J22 pad 56: /H2-24 -> /H1-52
- J22 pad 57: /H1-25 -> /+Y_SOLAR_TLE
- J22 pad 58: /H1-26 -> /-X_SOLAR_TLE
- J22 pad 59: 5V_SYS -> /+Y_SOLAR_PWR
- J22 pad 6: /+X_SOLAR_RTN -> /H1-2
- J22 pad 60: 5V_SYS -> /-X_SOLAR_PWR
- J22 pad 7: /-Z_SOLAR_PWR -> /H1-3
- J22 pad 8: /+X_SOLAR_PWR -> /H1-4
- J22 pad 9: /H1-1 -> /H1-5
- J23 pad 1: /H1-27 -> /-Z_SOLAR_TLE
- J23 pad 10: /5V_USB -> /H2-6
- J23 pad 11: /AGND -> /H2-7
- J23 pad 12: EP -> /H2-8
- J23 pad 13: V_RF -> /H2-9
- J23 pad 14: /H1-34 -> /H2-10
- J23 pad 15: /H2-33 -> /H2-11
- J23 pad 16: /H2-34 -> /H2-12
- J23 pad 17: /H1-35 -> /H2-13
- J23 pad 18: /H1-36 -> /H2-14
- J23 pad 19: /H2-35 -> /H2-15
- J23 pad 2: /H1-28 -> /+X_SOLAR_TLE
- J23 pad 20: /H2-36 -> /H2-16
- J23 pad 21: /H1-37 -> /H2-17
- J23 pad 22: /H1-38 -> /H2-18
- J23 pad 23: /H2-37 -> /H2-19
- J23 pad 24: /H2-38 -> /H2-20
- J23 pad 25: /H1-39 -> /H2-21
- J23 pad 26: /H1-40 -> /H2-22
- J23 pad 27: /H2-39 -> /H2-23
- J23 pad 28: /H2-40 -> /H2-24
- J23 pad 29: /H1-41 -> 5V_SYS
- J23 pad 3: 3.3V_SYS -> /-Z_SOLAR_PWR
- J23 pad 30: /H1-42 -> 5V_SYS
- J23 pad 31: /H2-41 -> 3.3V_SYS
- J23 pad 32: /H2-42 -> 3.3V_SYS
- J23 pad 33: /H1-43 -> GND
- J23 pad 34: /H1-44 -> GND
- J23 pad 35: /H2-43 -> /AGND
- J23 pad 36: /H2-44 -> GND
- J23 pad 37: /H1-45 -> /H2-33
- J23 pad 38: /H1-46 -> /H2-34
- J23 pad 39: VBATT -> /H2-35
- J23 pad 4: 3.3V_SYS -> /+X_SOLAR_PWR
- J23 pad 40: VBATT -> /H2-36
- J23 pad 41: /SELF_TEST -> /H2-37
- J23 pad 42: /USER_1 -> /H2-38
- J23 pad 43: EP -> /H2-39
- J23 pad 44: EP -> /H2-40
- J23 pad 45: /USER_2 -> /H2-41
- J23 pad 46: /USER_3 -> /H2-42
- J23 pad 47: VBATT_RET -> /H2-43
- J23 pad 48: VBATT_RET -> /H2-44
- J23 pad 49: /H1-51 -> VBATT
- J23 pad 5: /BUS_RESET -> /H2-1
- J23 pad 50: /H1-52 -> VBATT
- J23 pad 51: /H2-51 -> GND
- J23 pad 52: /H2-52 -> GND
- J23 pad 53: /+Y_SOLAR_TLE -> VBATT_RET
- J23 pad 54: /-X_SOLAR_TLE -> VBATT_RET
- J23 pad 55: /+Y_SOLAR_RTN -> /H2-51
- J23 pad 56: /-X_SOLAR_RTN -> /H2-52
- J23 pad 57: /+Y_SOLAR_PWR -> /+Y_SOLAR_RTN
- J23 pad 58: /-X_SOLAR_PWR -> /-X_SOLAR_RTN
- J23 pad 6: /H1-30 -> /H2-2
- J23 pad 7: EP -> /H2-3
- J23 pad 8: EP -> /H2-4
- J23 pad 9: /H1-31 -> /H2-5
- J7 pad 1: Net-(J7-Pad1) -> /+X_SOLAR_PWR
- J8 pad 1: Net-(J8-Pad1) -> /+X_SOLAR_RTN
- Q1 pad 2: EP -> GND
- Q10 pad 2: EP -> GND
- Q11 pad 2: EP -> GND
- Q12 pad 2: EP -> GND
- Q18 pad 2: EP -> GND
- Q19 pad 2: EP -> GND
- Q2 pad 2: EP -> GND
- Q22 pad 2: EP -> GND
- Q23 pad 2: EP -> GND
- Q3 pad 2: EP -> GND
- Q4 pad 2: EP -> GND
- Q5 pad 2: EP -> GND
- Q6 pad 2: EP -> GND
- Q7 pad 2: EP -> GND
- Q8 pad 2: EP -> GND
- Q9 pad 2: EP -> GND
- SW1 pad 3: EP -> GND
- SW2 pad 3: EP -> GND
- SW3 pad 3: EP -> GND
- SW4 pad 3: EP -> GND
- SW5 pad 3: EP -> GND
Routing:
- net GND: track 0.00 -> 8.05 mm, vias 0 -> 5
- net (no net): track 0.00 -> 7.35 mm, vias 0 -> 4
- net /RBF: track 8.57 -> 2.82 mm, vias 0 -> 1
- net /GND: track 5.37 -> 0.00 mm
- net VBATT_RET: track 0.00 -> 3.51 mm, vias 0 -> 2
- net VBATT: track 0.00 -> 3.51 mm, vias 0 -> 2
- net 5V_SYS: track 0.00 -> 3.51 mm, vias 0 -> 2
- net 3.3V_SYS: track 0.00 -> 3.02 mm, vias 0 -> 2
- net /H1-31: track 0.00 -> 2.82 mm, vias 0 -> 1
- net /H1-23: track 0.00 -> 2.82 mm, vias 0 -> 1
- net /SEP1: track 0.00 -> 2.82 mm, vias 0 -> 1
- net /H1-51: track 0.00 -> 2.82 mm, vias 0 -> 1
- net /H1-43: track 0.00 -> 2.82 mm, vias 0 -> 1
- net /H1-35: track 0.00 -> 2.82 mm, vias 0 -> 1
- net /H1-27: track 0.00 -> 2.82 mm, vias 0 -> 1
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Other:
- board outline removed
- copper layers 2 -> 6
- net class Default: clearance 0.2 -> 0.2032
- rule trace_clearance: 0.2 -> 0.2032

Commit message: 2
Parts:
- added H1: Conn_02x26_Odd_Even, Connector_PinHeader_2.54mm:PinHeader_2x26_P2.54mm_Vertical, F.Cu at (68.2, 90.2)
- added H2: Conn_02x26_Odd_Even, Connector_PinHeader_2.54mm:PinHeader_2x26_P2.54mm_Vertical, F.Cu at (73.2, 90.2)
- moved J4 208.0 mm to (261.6, 86.4)
- moved J9 206.6 mm to (261.6, 127.0)
- moved J15 202.5 mm to (261.6, 157.5)
- moved J16 202.4 mm to (261.6, 147.3)
- moved J17 202.4 mm to (261.6, 137.2)
- moved J13 202.2 mm to (261.6, 116.8)
- moved J18 202.2 mm to (261.6, 76.2)
- moved J7 202.2 mm to (261.6, 106.7)
- moved J11 202.2 mm to (261.6, 96.5)
- moved J21 172.0 mm to (243.8, 147.3)
- moved J19 171.9 mm to (243.8, 137.2)
- moved J10 171.9 mm to (243.8, 127.0)
- moved J3 171.8 mm to (241.3, 76.2), turned to 90 degrees
- moved J12 171.8 mm to (243.8, 116.8)
- moved J8 171.7 mm to (243.8, 106.7)
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Connections:
- SW1 pad 1: Net-(SW1-Pad1) -> unconnected-(SW1-Pad1)
- SW1 pad 2: Net-(SW1-Pad2) -> unconnected-(SW1-Pad2)
- SW2 pad 1: Net-(SW2-Pad1) -> unconnected-(SW2-Pad1)
- SW2 pad 2: Net-(SW2-Pad2) -> unconnected-(SW2-Pad2)
- SW3 pad 1: Net-(SW3-Pad1) -> unconnected-(SW3-Pad1)
- SW3 pad 2: Net-(SW3-Pad2) -> unconnected-(SW3-Pad2)
- SW4 pad 1: Net-(SW4-Pad1) -> unconnected-(SW4-Pad1)
- SW4 pad 2: Net-(SW4-Pad2) -> unconnected-(SW4-Pad2)
- SW5 pad 1: Net-(SW5-Pad1) -> unconnected-(SW5-Pad1)
- SW5 pad 2: Net-(SW5-Pad2) -> unconnected-(SW5-Pad2)
- SW6 pad 1: Net-(SW6-Pad1) -> unconnected-(SW6-Pad1)
- SW7 pad 1: Net-(SW7-Pad1) -> unconnected-(SW7-Pad1)
- SW8 pad 1: Net-(SW8-Pad1) -> unconnected-(SW8-Pad1)
- SW9 pad 1: Net-(SW9-Pad1) -> unconnected-(SW9-Pad1)
Routing:
- net GND: track 8.05 -> 20.3 mm, vias 5 -> 15
- net /H2-10: track 2.00 -> 10.3 mm, vias 1 -> 6
- net (no net): track 7.35 -> 0.00 mm, vias 4 -> 0
- net /H2-9: track 1.51 -> 8.52 mm, vias 1 -> 6
- net 5V_SYS: track 3.51 -> 8.47 mm, vias 2 -> 6
- net VBATT_RET: track 3.51 -> 8.47 mm, vias 2 -> 6
- net VBATT: track 3.51 -> 8.47 mm, vias 2 -> 6
- net 3.3V_SYS: track 3.02 -> 7.90 mm, vias 2 -> 6
- net /RBF: track 2.82 -> 5.31 mm, vias 1 -> 3
- net /H1-11: track 2.82 -> 5.31 mm, vias 1 -> 3
- net V_RF: track 1.51 -> 4.00 mm, vias 1 -> 3
- net /USER_2: track 1.51 -> 4.00 mm, vias 1 -> 3
- net /SELF_TEST: track 2.82 -> 5.31 mm, vias 1 -> 3
- net /H1-7: track 1.51 -> 4.00 mm, vias 1 -> 3
- net /H1-51: track 2.82 -> 5.31 mm, vias 1 -> 3
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Other:
- board outline added: 208 x 133.4 mm
- net class Default removed

Commit message: 1
Parts:
- turned J22 to -90 degrees
- turned J23 to -90 degrees
Routing:
- net /+X_SOLAR_RTN: track 3.95 -> 33.7 mm
- net /H1-8: track 3.95 -> 33.4 mm
- net /H1-12: track 3.95 -> 33.1 mm
- net /H1-16: track 3.95 -> 32.8 mm
- net /H1-4: track 3.95 -> 32.7 mm
- net /H1-20: track 3.95 -> 32.6 mm
- net /H1-52: track 3.95 -> 32.5 mm
- net /-X_SOLAR_PWR: track 3.95 -> 32.3 mm
- net /H1-24: track 3.95 -> 32.3 mm
- net /H1-28: track 3.95 -> 32.0 mm
- net /USER_1: track 3.95 -> 31.9 mm
- net /H1-44: track 3.95 -> 31.6 mm
- net /H1-40: track 3.95 -> 31.3 mm
- net /H1-10: track 2.48 -> 29.7 mm, vias 2 -> 3
- net /H1-36: track 3.95 -> 31.0 mm
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
Commit message: 1
Parts:
- turned J22 to 90 degrees
- turned J23 to 90 degrees
Routing:
- net GND: track 21.5 -> 354.5 mm
- net 3.3V_SYS: track 8.06 -> 146.4 mm
- net VBATT_RET: track 8.47 -> 141.8 mm
- net 5V_SYS: track 8.43 -> 141.5 mm
- net VBATT: track 8.47 -> 141.1 mm
- net /H2-1: track 6.31 -> 93.0 mm
- net /H2-51: track 4.03 -> 82.1 mm
- net /H2-5: track 3.84 -> 79.7 mm
- net /H2-7: track 4.03 -> 79.5 mm
- net /H2-9: track 3.99 -> 79.3 mm
- net /H2-13: track 3.99 -> 79.2 mm
- net /H2-17: track 3.99 -> 79.2 mm
- net /H2-15: track 4.03 -> 79.0 mm
- net /H2-11: track 4.03 -> 79.0 mm
- net /H2-41: track 3.99 -> 78.9 mm
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
Commit message: 1
Parts:
- moved H1 233.7 mm to (294.2, 149.8), turned to 180 degrees
- moved H2 224.0 mm to (289.1, 149.8), turned to 180 degrees
- moved J11 188.4 mm to (73.3, 102.4)
- moved J13 188.4 mm to (73.3, 122.7)
- moved J15 188.4 mm to (73.3, 163.4)
- moved J16 188.4 mm to (73.3, 153.2)
- moved J17 188.4 mm to (73.3, 143.1)
- moved J18 188.4 mm to (73.3, 82.1)
- moved J4 188.4 mm to (73.3, 92.2)
- moved J7 188.4 mm to (73.3, 112.6)
- moved J9 188.4 mm to (73.3, 132.9)
- moved D22 180.8 mm to (76.2, 180.7)
- moved Q23 180.8 mm to (76.2, 176.3)
- moved R36 177.0 mm to (78.1, 180.7)
- moved R39 175.7 mm to (78.7, 176.3)
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Routing:
- net GND: track 354.5 -> 997.1 mm
- net /+Y_SOLAR_PWR: track 21.1 -> 390.8 mm
- net /H1-35: track 58.4 -> 420.0 mm
- net /+Y_SOLAR_TLE: track 20.6 -> 370.5 mm
- net /H1-51: track 58.9 -> 389.6 mm
- net /USER_2: track 55.9 -> 371.7 mm
- net /SELF_TEST: track 58.7 -> 358.4 mm
- net /H1-45: track 55.1 -> 347.2 mm
- net /H1-43: track 59.0 -> 323.2 mm
- net 3.3V_SYS: track 146.4 -> 406.4 mm
- net 5V_SYS: track 141.5 -> 394.8 mm
- net /H1-41: track 54.8 -> 302.7 mm
- net VBATT_RET: track 141.8 -> 377.4 mm
- net /H1-39: track 59.0 -> 289.3 mm
- net /RBF: track 59.7 -> 278.5 mm
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Other:
- board size 208 x 133.4 mm -> 224.9 x 138.5 mm
- board text added: "H2-1"

Commit message: 1
Parts:
- removed J3: DEBUG POWER SEND JUMPER, Connector_PinHeader_2.54mm:PinHeader_1x02_P2.54mm_Vertical
Connections:
- H1 pad 32: /5V_USB -> 5V_DEBUG
- J1 pad 36: /5V_USB -> 5V_DEBUG
- J200_1 pad 70: /5V_USB -> 5V_DEBUG
- J22 pad 36: /5V_USB -> 5V_DEBUG
- TP70 pad 1: /5V_USB -> 5V_DEBUG
Routing:
- net GND: track 997.1 -> 1563.1 mm
- net 5V_DEBUG: track 0.00 -> 407.2 mm, vias 0 -> 3
- net 3.3V_SYS: track 406.4 -> 690.5 mm
- net 5V_SYS: track 394.8 -> 664.2 mm
- net /H1-16: track 194.4 -> 445.6 mm
- net /H1-36: track 196.6 -> 439.5 mm
- net /H1-14: track 185.7 -> 426.4 mm
- net /H1-12: track 177.8 -> 413.9 mm
- net /H1-13: track 179.7 -> 412.8 mm
- net /H1-34: track 186.7 -> 419.5 mm
- net /-X_SOLAR_PWR: track 175.1 -> 402.8 mm
- net /H1-10: track 171.8 -> 397.3 mm
- net /H1-8: track 161.9 -> 384.4 mm
- net V_RF: track 181.8 -> 404.0 mm
- net /H1-9: track 164.7 -> 383.8 mm
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