File: backplane-boards/backplane-breakout-big/backplane-breaout-big.kicad_sch (KiCad schematic)
At the start: 241 parts, among them J1 Breakout Connector, J10 -Z_SOLAR_RTN, J11 +Y_SOLAR_PWR, J12 +Y_SOLAR_RTN, J13 -X_SOLAR_PWR, J14 -X_SOLAR_RTN, J15 3.3V_SYS, J16 +5V_SYS, J17 VCC_RF, J18 5V_DEBUG, J19 GND, J2 Breakout Connector, J20 Conn_02x04_Odd_Even, J200_1 HSEC8-160-01-S-DV-A-K-TR, J21 AGND, J22 SSM-130-L-DV, J23 SSM-130-L-DV, J24 GND, J3 DEBUG POWER SEND JUMPER, J4 PACK+, J5 Conn_01x08, J6 PACK-, J7 +X_SOLAR_PWR, J8 +X_SOLAR_RTN, J9 -Z_SOLAR_PWR, Q1 DMG1012UW-7, Q10 DMG1012UW-7, Q11 DMG1012UW-7, Q12 DMG1012UW-7, Q13 BSS84W-7-F, Q14 BSS84W-7-F, Q15 BSS84W-7-F, Q16 BSS84W-7-F, Q17 BSS84W-7-F, Q18 DMG1012UW-7, Q19 DMG1012UW-7, Q2 DMG1012UW-7, Q20 BSS84W-7-F, Q21 BSS84W-7-F, Q22 DMG1012UW-7, Q23 DMG1012UW-7, Q3 DMG1012UW-7, Q4 DMG1012UW-7, Q5 DMG1012UW-7, Q6 DMG1012UW-7, Q7 DMG1012UW-7, Q8 DMG1012UW-7, Q9 DMG1012UW-7, SW1 SEP1, SW2 SEP2, SW3 SEP3, SW4 SEP4, SW5 RBF, SW6 USER_SW_1, SW7 USER_SW_2, SW8 USER_SW_3, SW9 USER_SW_4

Commit message: 1
Parts:
- removed J3: DEBUG POWER SEND JUMPER, Connector_PinHeader_2.54mm:PinHeader_1x02_P2.54mm_Vertical, symbol Connector_Generic:Conn_01x02
Connections:
- net 5V_USB is gone; now on net 5V_DEBUG: H1.32 (Pin_32), J1.36 (Pin_36), J200_1.70 (Pin_70), J22.36 (Pin_36), TP70.1
Other:
- note removed: "connecting this will send 5V debug to the backplane"
Changed lines of the file:
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@@
     (stroke (width 0) (type default) (color 0 0 0 0))
   )
-  (wire (pts (xy 228.6 31.75) (xy 228.6 33.02))
-    (stroke (width 0) (type default) (color 0 0 0 0))
-  )
   (wire (pts (xy 303.53 308.61) (xy 327.66 308.61))
     (stroke (width 0) (type default) (color 0 0 0 0))
@@
     (stroke (width 0) (type default) (color 0 0 0 0))
   )
-  (wire (pts (xy 228.6 35.56) (xy 228.6 36.83))
-    (stroke (width 0) (type default) (color 0 0 0 0))
-  )
   (wire (pts (xy 488.696 298.45) (xy 449.58 298.45))
     (stroke (width 0) (type default) (color 0 0 0 0))
@@
     (stroke (width 0) (type default) (color 0 0 0 0))
   )
-  (wire (pts (xy 215.9 33.02) (xy 228.6 33.02))
-    (stroke (width 0) (type default) (color 0 0 0 0))
-  )
   (wire (pts (xy 219.456 257.81) (xy 180.34 257.81))
     (stroke (width 0) (type default) (color 0 0 0 0))
@@
     (stroke (width 0) (type default) (color 0 0 0 0))
   )
-  (wire (pts (xy 488.696 300.99) (xy 449.58 300.99))
+  (wire (pts (xy 167.64 168.91) (xy 175.26 168.91))
     (stroke (width 0) (type default) (color 0 0 0 0))
   )
-  (wire (pts (xy 215.9 35.56) (xy 228.6 35.56))
+  (wire (pts (xy 488.696 300.99) (xy 449.58 300.99))
     (stroke (width 0) (type default) (color 0 0 0 0))
   )
@@
     (effects (font (size 1.524 1.524)) (justify left bottom))
   )
-  (text "connecting this will send 5V debug to the backplane"
-    (at 201.93 24.13 0)
-    (effects (font (size 1.27 1.27)) (justify left bottom))
-  )
   (text "GND header to grab ground" (at 158.75 405.13 0)
     (effects (font (size 1.27 1.27)) (justify left bottom))
@@
     (effects (font (size 1.524 1.524)) (justify left bottom))
   )
-  (label "5V_USB" (at 228.6 31.75 0)
-    (effects (font (size 1.524 1.524)) (justify left bottom))
-  )
   (label "H2-27" (at 137.16 133.35 0)
     (effects (font (size 1.524 1.524)) (justify left bottom))
@@
     (effects (font (size 1.524 1.524)) (justify left bottom))
   )
+  (label "5V_USB" (at 175.26 168.91 0)
+    (effects (font (size 1.524 1.524)) (justify left bottom))
+  )
   (label "H2-20" (at 472.44 336.55 0)
     (effects (font (size 1.524 1.524)) (justify left bottom))
@@
     (effects (font (size 1.524 1.524)) (justify left bottom))
   )
+  (label "5V_USB" (at 138.43 168.91 0)
+    (effects (font (size 1.524 1.524)) (justify left bottom))
+  )
   (label "H2-3" (at 406.4 316.23 0)
     (effects (font (size 1.524 1.524)) (justify left bottom))
@@
     (effects (font (size 1.524 1.524)) (justify left bottom))
   )
+  (global_label "5V_DEBUG" (shape input) (at 167.64 168.91 180) (fields_autoplaced)
+    (effects (font (size 1.27 1.27)) (justify right))
+    (property "Intersheet References" "${INTERSHEET_REFS}" (id 0) (at -133.35 138.43 0)
+      (effects (font (size 1.27 1.27)) hide)
+    )
+  )
   (global_label "V_RF" (shape input) (at 331.47 77.47 180) (fields_autoplaced)
     (effects (font (size 1.27 1.27)) (justify right))
@@
     )
   )
-  (global_label "5V_DEBUG" (shape input) (at 228.6 36.83 0) (fields_autoplaced)
-    (effects (font (size 1.27 1.27)) (justify left))
-    (property "Intersheet References" "${INTERSHEET_REFS}" (id 0) (at 0 0 0)
-      (effects (font (size 1.27 1.27)) hide)
-    )
-  )
-  (global_label "5V_DEBUG" (shape input) (at 138.43 168.91 0) (fields_autoplaced)
-    (effects (font (size 1.27 1.27)) (justify left))
-    (property "Intersheet References" "${INTERSHEET_REFS}" (id 0) (at 0 0 0)
-      (effects (font (size 1.27 1.27)) hide)
-    )
-  )
   (global_label "5V_DEBUG" (shape input) (at 508 156.21 180) (fields_autoplaced)
     (effects (font (size 1.27 1.27)) (justify right))
@@
     (pin "9")
   )
-  (symbol (lib_id "Connector_Generic:Conn_01x02") (at 210.82 33.02 0) (mirror y) (unit 1)
-    (in_bom yes) (on_board yes)
-    (property "Reference" "J3" (id 0) (at 212.9028 27.5082 0))
-    (property "Value" "DEBUG POWER SEND JUMPER" (id 1) (at 212.9028 29.8196 0))
-    (property "Footprint" "Connector_PinHeader_2.54mm:PinHeader_1x02_P2.54mm_Vertical" (id 2) (at 210.82 33.02 0)
-      (effects (font (size 1.27 1.27)) hide)
-    )
-    (property "Datasheet" "~" (id 3) (at 210.82 33.02 0)
-      (effects (font (size 1.27 1.27)) hide)
-    )
-    (pin "1")
-    (pin "2")
-  )
   (symbol (lib_id "Switch:SW_SPDT") (at 223.52 45.72 0) (unit 1)
     (in_bom yes) (on_board yes)
@@
     (pin "1")
   )
-  (symbol (lib_id "backplane-breakout-big:Conn_02x60_Top_Bottom") (at 58.42 227.33 0)
+  (symbol (lib_id "backplane-breakout-big:Conn_02x60_Top_Bottom") (at 58.42 227.33 0) (unit 1)
     (in_bom yes) (on_board yes)
     (property "Reference" "J200_1" (id 0) (at 58.42 223.0882 0))
@@
       (reference "J2") (unit 1) (value "Breakout Connector") (footprint "backplane-breakout-big:SAMTEC_FTSH-130-04-L-DH_flipped")
     )
-    (path "/00000000-0000-0000-0000-000061e53516"
-      (reference "J3") (unit 1) (value "DEBUG POWER SEND JUMPER") (footprint "Connector_PinHeader_2.54mm:PinHeader_1x02_P2.54mm_Vertical")
-    )
     (path "/00000000-0000-0000-0000-000061d27792"

Commit message: routed more
Parts:
- removed J10: -Z_SOLAR_RTN, backplane-breakout-big:Keystone_476, symbol Connector_Generic:Conn_01x01
- removed J11: +Y_SOLAR_PWR, backplane-breakout-big:Keystone_476, symbol Connector_Generic:Conn_01x01
- removed J12: +Y_SOLAR_RTN, backplane-breakout-big:Keystone_476, symbol Connector_Generic:Conn_01x01
- removed J13: -X_SOLAR_PWR, backplane-breakout-big:Keystone_476, symbol Connector_Generic:Conn_01x01
- removed J14: -X_SOLAR_RTN, backplane-breakout-big:Keystone_476, symbol Connector_Generic:Conn_01x01
- removed J15: 3.3V_SYS, backplane-breakout-big:Keystone_476, symbol Connector_Generic:Conn_01x01
- removed J16: +5V_SYS, backplane-breakout-big:Keystone_476, symbol Connector_Generic:Conn_01x01
- removed J17: VCC_RF, backplane-breakout-big:Keystone_476, symbol Connector_Generic:Conn_01x01
- removed J21: AGND, backplane-breakout-big:Keystone_476, symbol Connector_Generic:Conn_01x01
- removed J4: PACK+, backplane-breakout-big:Keystone_476, symbol Connector_Generic:Conn_01x01
- removed J6: PACK-, backplane-breakout-big:Keystone_476, symbol Connector_Generic:Conn_01x01
- removed J7: +X_SOLAR_PWR, backplane-breakout-big:Keystone_476, symbol Connector_Generic:Conn_01x01
- removed J8: +X_SOLAR_RTN, backplane-breakout-big:Keystone_476, symbol Connector_Generic:Conn_01x01
- removed J9: -Z_SOLAR_PWR, backplane-breakout-big:Keystone_476, symbol Connector_Generic:Conn_01x01
- added SW10: BUS_RESET, backplane-breakout-big:SW_2-1437565-9, symbol Switch:SW_SPST
- added SW11: SELF_TEST, backplane-breakout-big:SW_2-1437565-9, symbol Switch:SW_SPST
Connections:
- net USER_SW_1 is gone; now on net USER_SW_1_SEND: SW6.2 (B)
- net USER_SW_2 is gone; now on net USER_SW_2_SEND: SW7.2 (B)
- net USER_SW_3 is gone; now on net USER_SW_3_SEND: SW8.2 (B)
- net USER_SW_4 is gone; now on net USER_SW_4_SEND: SW9.2 (B)
- net BUS_RESET: now also SW10.1 (A)
- net GND: now also SW10.2 (B), SW11.2 (B)
- net RBF: now also SW5.2 (B)
- net SELF_TEST: now also SW11.1 (A)
- net SEP1: now also SW1.2 (B)
- net SEP2: now also SW2.2 (B)
- net SEP3: now also SW3.2 (B)
- net SEP4: now also SW4.2 (B)
- net VBATT: no longer H2.45 (Pin_45), H2.46 (Pin_46), J2.49 (Pin_49), J2.50 (Pin_50), J200_1.100 (Pin_100), J200_1.99 (Pin_99), J23.49 (Pin_49), J23.50 (Pin_50), TP100.1, TP99.1
- net V_RF: no longer H1.33 (Pin_33), J1.37 (Pin_37), J200_1.73 (Pin_73), J22.37 (Pin_37), TP73.1
- net 3.3V_SYS renamed H2-27
- net H2-27: no longer H2.28 (Pin_28), J2.32 (Pin_32), J200_1.64 (Pin_64), J23.32 (Pin_32), TP64.1
- net 5V_SYS renamed H2-25
- net H2-25: no longer H2.26 (Pin_26), J2.30 (Pin_30), J200_1.60 (Pin_60), J23.30 (Pin_30), TP60.1
- net USER_1 renamed H1-48
- net USER_2 renamed H1-49
- net USER_3 renamed H1-50
- net VBATT_RET renamed H2-49
- net H2-49: no longer H2.50 (Pin_50), J2.54 (Pin_54), J200_1.108 (Pin_108), J23.54 (Pin_54), TP108.1
- new net H1-33: H1.33 (Pin_33), J1.37 (Pin_37), J200_1.73 (Pin_73), J22.37 (Pin_37), TP73.1
- new net H2-26: H2.26 (Pin_26), J2.30 (Pin_30), J200_1.60 (Pin_60), J23.30 (Pin_30), TP60.1
- new net H2-28: H2.28 (Pin_28), J2.32 (Pin_32), J200_1.64 (Pin_64), J23.32 (Pin_32), TP64.1
- new net H2-45: H2.45 (Pin_45), J2.49 (Pin_49), J200_1.99 (Pin_99), J23.49 (Pin_49), TP99.1
- new net H2-46: H2.46 (Pin_46), J2.50 (Pin_50), J200_1.100 (Pin_100), J23.50 (Pin_50), TP100.1
- new net H2-50: H2.50 (Pin_50), J2.54 (Pin_54), J200_1.108 (Pin_108), J23.54 (Pin_54), TP108.1
Other:
- note added: "5V debug"
- note added: "BUTTONS"
- note removed: "POWER DELIVERY + MEASUREMENT"
- moved on the sheet: J18, J19, J20, SW1, SW2, SW3, SW4, SW5, SW6, SW7, SW8, SW9

Commit message: completion push
Parts:
- removed J18: 5V_DEBUG, backplane-breakout-big:Keystone_476, symbol Connector_Generic:Conn_01x01
- removed J19: GND, backplane-breakout-big:Keystone_476, symbol Connector_Generic:Conn_01x01
- added H5, H6, H7, H8: M3 HOLE, MountingHole:MountingHole_3.2mm_M3_Pad_TopBottom, symbol Mechanical:MountingHole_Pad
- J6: renamed from J20; value Conn_02x04_Odd_Even -> USER_SW
- J7: renamed from J5; value Conn_01x08 -> USER_LEDs
- TP109: renamed from TP98; value VBATT+ (H1-46) -> VBATT+
- TP111: renamed from TP102; value USER_1 (H1-48) -> H1-48
- TP112: renamed from TP104; value GND (H2-48) -> GND
- TP113: renamed from TP106; value USER_3 (H1-50) -> H1-50
- TP114: renamed from TP108; value VBATT- (H2-50) -> VBATT-
- TP115: renamed from TP110; value USER_5 (H1-52) -> H1-52
- TP116: renamed from TP112; value USER_11 (H2-52) -> H2-52
- TP19: renamed from TP37; value RBF (H1-15) -> RBF
- TP30: renamed from TP59; value 5V_SYS (H2-25) -> 5V_SYS
- TP32: renamed from TP63; value 3.3V_SYS (H2-27) -> 3.3V_SYS
- TP33: renamed from TP65; value ~RESET~ (H1-29) -> ~RESET~
- TP34: renamed from TP67; value GND (H2-29) -> GND
- TP36: renamed from TP71; value AGND (H2-31) -> AGND
- TP37: renamed from TP73; value VCC_RF (H1-33) -> RF_VCC
- TP45: renamed from TP89; value H1-41 -> SDA_SYS
- TP47: renamed from TP93; value H1-43 -> SCL_SYS
- TP49: renamed from TP97; value VBATT+ (H2-45) -> VBATT+
- TP50: renamed from TP99; value USER_6 (H2-45) -> H2-45
- TP51: renamed from TP101; value SELF_TEST (H1-47) -> SELF_TEST
- TP52: renamed from TP103; value GND (H2-47) -> GND
- TP53: renamed from TP105; value USER_2 (H1-49) -> H1-49
- TP54: renamed from TP107; value VBATT- (H2-49) -> VBATT-
- TP55: renamed from TP109; value USER_4 (H1-51) -> H1-51
- TP56: renamed from TP111; value USER_10 (H2-51) -> H2-51
- TP90: renamed from TP60; value 5V_SYS (H2-26) -> 5V_SYS
- TP92: renamed from TP64; value 3.3V_SYS (H2-28) -> 3.3V_SYS
- TP94: renamed from TP68; value GND (H2-30) -> GND
- TP95: renamed from TP70; value 5V_USB (H1-32) -> 5V_USB
- TP96: renamed from TP72; value GND (H2-32) -> GND
- renumbered D15 to D1, D18 to D10, D3 to D11, D9 to D12, D19 to D13, D5 to D14, D10 to D15, D20 to D16, D4 to D17, D11 to D18, D13 to D19, D1 to D2, D6 to D20, D12 to D21, D14 to D22, D22 to D23, D7 to D3, D21 to D4, D16 to D5, D23 to D6, D2 to D7, D17 to D9, J2 to J1, J1 to J2, J24 to J3, J22 to J4, J23 to J5, J200_1 to J8, Q13 to Q1, Q16 to Q10, Q3 to Q11, Q9 to Q12, Q17 to Q13, Q5 to Q14, Q10 to Q15, Q22 to Q16, Q4 to Q17, Q11 to Q18, Q18 to Q19, Q1 to Q2, Q6 to Q20, Q12 to Q21, Q19 to Q22, Q7 to Q3, Q20 to Q4, Q14 to Q5, Q21 to Q6, Q2 to Q7, Q15 to Q9, R7 to R1, R37 to R10, R2 to R11, R14 to R12, R29 to R13, R9 to R14, R21 to R15, R30 to R16, R3 to R17, R15 to R18, R31 to R19, R19 to R2, R11 to R20, R22 to R21, R5 to R22, R16 to R23, R38 to R24, R10 to R25, R23 to R26, R32 to R27, R34 to R28, R4 to R29, R27 to R3, R17 to R30, R25 to R31, R12 to R32, R24 to R33, R33 to R34, R39 to R35, R6 to R36, R18 to R37, R26 to R38, R36 to R39, R1 to R4, R13 to R5, R35 to R6, R28 to R7, R20 to R9, SW10 to SW1, SW4 to SW10, SW5 to SW11, SW11 to SW2, SW6 to SW3, SW7 to SW4, SW8 to SW5, SW9 to SW6, SW1 to SW7, SW2 to SW8, SW3 to SW9, TP19 to TP10, TP80 to TP100, TP82 to TP101, TP84 to TP102, TP86 to TP103, TP88 to TP104, TP90 to TP105, TP92 to TP106, TP94 to TP107, TP96 to TP108, TP21 to TP11, TP100 to TP110, TP114 to TP117, TP116 to TP118, TP118 to TP119, TP23 to TP12, TP25 to TP13, TP27 to TP14, TP29 to TP15, TP31 to TP16, TP33 to TP17, TP35 to TP18, TP3 to TP2, TP39 to TP20, TP41 to TP21, TP43 to TP22, TP45 to TP23, TP47 to TP24, TP49 to TP25, TP51 to TP26, TP53 to TP27, TP55 to TP28, TP57 to TP29, TP5 to TP3, TP61 to TP31, TP69 to TP35, TP75 to TP38, TP77 to TP39, TP7 to TP4, TP79 to TP40, TP81 to TP41, TP83 to TP42, TP85 to TP43, TP87 to TP44, TP91 to TP46, TP95 to TP48, TP9 to TP5, TP113 to TP57, TP115 to TP58, TP117 to TP59, TP11 to TP6, TP119 to TP60, TP2 to TP61, TP4 to TP62, TP6 to TP63, TP8 to TP64, TP10 to TP65, TP12 to TP66, TP14 to TP67, TP16 to TP68, TP18 to TP69, TP13 to TP7, TP20 to TP70, TP22 to TP71, TP24 to TP72, TP26 to TP73, TP28 to TP74, TP30 to TP75, TP32 to TP76, TP34 to TP77, TP36 to TP78, TP38 to TP79, TP15 to TP8, TP40 to TP80, TP42 to TP81, TP44 to TP82, TP46 to TP83, TP48 to TP84, TP50 to TP85, TP52 to TP86, TP54 to TP87, TP56 to TP88, TP58 to TP89, TP17 to TP9, TP62 to TP91, TP66 to TP93, TP74 to TP97, TP76 to TP98, TP78 to TP99
Connections:
- net VBATT is gone; now on net H2-26: Q12.1 (G), R15.1
- net V_PLD is gone; now on net H1-33: Q15.1 (G), R21.1
- net V_RF is gone; now on net H2-27: Q8.1 (G), R9.1
- no-connect marks 7 -> 11
Other:
- note added: "3.3v_SYS"
- note added: "5v_SYS"
- note added: "RF_vcc"
- note removed: "5V debug"
- note removed: "POWER ENTRY MINI-NANA JACKS"

Commit message: 1
Other:
- note added: "CSK (PC/104) BUS CONNECTOR"
- note added: "INDICATOR LEDs"
- note added: "MOUNTING HOLES"
- note added: "USER LEDs"
- note removed: "CSK BUS CONNECTOR"
- note removed: "DISCRETE INDICATOR LEDs"
- note removed: "DISCRETE USER LEDs"
- moved on the sheet: SW1, SW2

Commit message: fab files generated 2 pcbway
Parts:
- added H10, H11, H9: M3 HOLE, MountingHole:MountingHole_3.2mm_M3_Pad_TopBottom, symbol Mechanical:MountingHole_Pad
- H1, H2: value Conn_02x26_Odd_Even -> ESQ-132-12-G-D
Connections:
- no-connect marks 11 -> 14
Changed lines of the file:
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@@
   (no_connect (at 149.86 154.94))
   (no_connect (at 233.68 97.79))
+  (no_connect (at 176.53 173.99))
   (no_connect (at 233.68 25.4))
   (no_connect (at 231.14 124.46))
+  (no_connect (at 176.53 163.83))
   (no_connect (at 163.83 154.94))
   (no_connect (at 233.68 58.42))
   (no_connect (at 231.14 111.76))
   (no_connect (at 233.68 78.74))
+  (no_connect (at 176.53 154.94))
   (no_connect (at 163.83 163.83))
   (no_connect (at 149.86 163.83))
@@
     (in_bom yes) (on_board yes) (fields_autoplaced)
     (property "Reference" "H1" (id 0) (at 443.23 234.7935 0))
-    (property "Value" "Conn_02x26_Odd_Even" (id 1) (at 443.23 237.5686 0))
+    (property "Value" "ESQ-132-12-G-D" (id 1) (at 443.23 237.5686 0))
     (property "Footprint" "Connector_PinHeader_2.54mm:PinHeader_2x26_P2.54mm_Vertical" (id 2) (at 441.96 270.51 0)
       (effects (font (size 1.27 1.27)) hide)
@@
     (pin "1")
   )
+  (symbol (lib_id "Mechanical:MountingHole_Pad") (at 173.99 154.94 90) (unit 1)
+    (in_bom yes) (on_board yes) (fields_autoplaced)
+    (property "Reference" "H9" (id 0) (at 172.72 147.32 90)
+      (effects (font (size 1.27 1.27)) hide)
+    )
+    (property "Value" "M3 HOLE" (id 1) (at 172.72 149.86 90))
+    (property "Footprint" "MountingHole:MountingHole_3.2mm_M3_Pad_TopBottom" (id 2) (at 173.99 154.94 0)
+      (effects (font (size 1.27 1.27)) hide)
+    )
+    (property "Datasheet" "~" (id 3) (at 173.99 154.94 0)
+      (effects (font (size 1.27 1.27)) hide)
+    )
+    (pin "1")
+  )
   (symbol (lib_id "Connector_Generic:Conn_02x26_Odd_Even") (at 441.96 344.17 0) (unit 1)
     (in_bom yes) (on_board yes) (fields_autoplaced)
     (property "Reference" "H2" (id 0) (at 443.23 308.4535 0))
-    (property "Value" "Conn_02x26_Odd_Even" (id 1) (at 443.23 311.2286 0))
+    (property "Value" "ESQ-132-12-G-D" (id 1) (at 443.23 311.2286 0))
     (property "Footprint" "Connector_PinHeader_2.54mm:PinHeader_2x26_P2.54mm_Vertical" (id 2) (at 441.96 344.17 0)
       (effects (font (size 1.27 1.27)) hide)
@@
     (pin "1")
   )
+  (symbol (lib_id "Mechanical:MountingHole_Pad") (at 173.99 173.99 90) (unit 1)
+    (in_bom yes) (on_board yes) (fields_autoplaced)
+    (property "Reference" "H11" (id 0) (at 172.72 166.37 90)
+      (effects (font (size 1.27 1.27)) hide)
+    )
+    (property "Value" "M3 HOLE" (id 1) (at 172.72 168.91 90))
+    (property "Footprint" "MountingHole:MountingHole_3.2mm_M3_Pad_TopBottom" (id 2) (at 173.99 173.99 0)
+      (effects (font (size 1.27 1.27)) hide)
+    )
+    (property "Datasheet" "~" (id 3) (at 173.99 173.99 0)
+      (effects (font (size 1.27 1.27)) hide)
+    )
+    (pin "1")
+  )
   (symbol (lib_id "Switch:SW_SPST") (at 152.4 40.64 0) (unit 1)
     (in_bom yes) (on_board yes)
@@
     (pin "1")
   )
+  (symbol (lib_id "Mechanical:MountingHole_Pad") (at 173.99 163.83 90) (unit 1)
+    (in_bom yes) (on_board yes) (fields_autoplaced)
+    (property "Reference" "H10" (id 0) (at 172.72 156.21 90)
+      (effects (font (size 1.27 1.27)) hide)
+    )
+    (property "Value" "M3 HOLE" (id 1) (at 172.72 158.75 90))
+    (property "Footprint" "MountingHole:MountingHole_3.2mm_M3_Pad_TopBottom" (id 2) (at 173.99 163.83 0)
+      (effects (font (size 1.27 1.27)) hide)
+    )
+    (property "Datasheet" "~" (id 3) (at 173.99 163.83 0)
+      (effects (font (size 1.27 1.27)) hide)
+    )
+    (pin "1")
+  )
   (sheet_instances
     (path "/" (page "1"))
@@
     )
     (path "/843cf889-0d60-4c94-8d29-d8b862da10fd"
-      (reference "H1") (unit 1) (value "Conn_02x26_Odd_Even") (footprint "Connector_PinHeader_2.54mm:PinHeader_2x26_P2.54mm_Vertical")
+      (reference "H1") (unit 1) (value "ESQ-132-12-G-D") (footprint "Connector_PinHeader_2.54mm:PinHeader_2x26_P2.54mm_Vertical")
     )
     (path "/98bb8986-76a0-4b47-9788-977a2f2abfd2"
-      (reference "H2") (unit 1) (value "Conn_02x26_Odd_Even") (footprint "Connector_PinHeader_2.54mm:PinHeader_2x26_P2.54mm_Vertical")
+      (reference "H2") (unit 1) (value "ESQ-132-12-G-D") (footprint "Connector_PinHeader_2.54mm:PinHeader_2x26_P2.54mm_Vertical")
     )
     (path "/dd79a151-a567-4948-ad49-91cc4a85664e"
@@
       (reference "H8") (unit 1) (value "M3 HOLE") (footprint "MountingHole:MountingHole_3.2mm_M3_Pad_TopBottom")
     )
+    (path "/915da06d-fd1f-4007-b9e4-aa3b51a560b3"
+      (reference "H9") (unit 1) (value "M3 HOLE") (footprint "MountingHole:MountingHole_3.2mm_M3_Pad_TopBottom")
+    )
+    (path "/f624f850-ac4f-4447-a510-d3bc414cb6b2"
+      (reference "H10") (unit 1) (value "M3 HOLE") (footprint "MountingHole:MountingHole_3.2mm_M3_Pad_TopBottom")
+    )
+    (path "/ba7195ae-a1f4-4965-82ea-89d705092be4"
+      (reference "H11") (unit 1) (value "M3 HOLE") (footprint "MountingHole:MountingHole_3.2mm_M3_Pad_TopBottom")
+    )
     (path "/00000000-0000-0000-0000-000061e5281c"
