File: backplane.sch (KiCad schematic (older format))
At the start: 32 parts, among them J101 BURN_WIRES, J102 -Z SOLAR PANEL, J103 SEP1 & SEP2, J104 SEP3 & SEP4, J105 +X SOLAR PANEL, J106 -X SOLAR PANEL, J107 +Y SOLAR PANEL, J200_1 HSEC8-160-01-S-DV-A-K-TR, J200_2 HSEC8-160-01-S-DV-A-K-TR, J200_3 HSEC8-160-01-S-DV-A-K-TR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

Commit message: rbf
Other:
- note added: "breakout connectors are spaced such that the breakout thickness is 3.2mm!!"
Changed lines of the file:
@@
 Text Label 17150 3950 0    60   ~ 0
 CHS
+Text Notes 15200 13000 0    100  ~ 0
+breakout connectors are spaced such that the breakout thickness is 3.2mm!!
 $EndSCHEMATC
