File: backplane-boards/backplane-rbf/backplane-rbf.sch (KiCad schematic (older format))
At the start: 3 parts, among them J1 Breakout Connector, J2 Breakout Connector

Commit message: rbf
Parts:
- removed J1, J2: Breakout Connector, backplane-rbf:SAMTEC_LSH-030-01-X-D-A-TR, symbol Connector_Generic:Conn_02x30_Odd_Even
- added J300, J301: FTS-130-01-L-SV, backplane-rbf:FTS-130-01-L-SV, symbol Connector_Generic:Conn_01x30
Connections:
- net labels removed: +X_SOLAR_RTN, +Y_SOLAR_RTN, -X_SOLAR_PWR, -X_SOLAR_TLE, -Z_SOLAR_PWR, -Z_SOLAR_TLE, 5V_USB, AGND, H1-10, H1-12, H1-14, H1-16, H1-18, H1-2, H1-20, H1-22, H1-24, H1-26, H1-28, H1-30, H1-34, H1-36, H1-38, H1-4, H1-40, H1-42, H1-44, H1-46, H1-52, H1-6, H1-8, H2-1, H2-11, H2-13, H2-15, H2-17, H2-19, H2-21, H2-23, H2-25, H2-27, H2-3, H2-33, H2-35, H2-37, H2-39, H2-41, H2-43, H2-45, H2-49, H2-5, H2-51, H2-7, H2-9, SEP2, SEP3, USER_1, USER_3
- wire segments 122 -> 62
